File: IoTmanager/IoTmanager.kicad_pcb (KiCad board)
At the start: 2 copper layers, 41 parts, among them J1 Program-connector, K1 ZC32F-012-HS3-copy, K2 ZC32F-012-HS3-copy, K3 ZC32F-012-HS3-copy, K4 ZC32F-012-HS3-copy, Q1 BC817, Q2 BC817, Q3 BC817, Q4 BC817, U2 ESP-12F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

Commit message: update
Parts:
- removed Flash1: SW_Omron_B3FS, Button_Switch_SMD:SW_SPST_Omron_B3FS-100xP
- removed K3: ZC32F-012-HS3-copy, module-custom-for-esp8266:ZC32F-012-HS3
- removed R4, R7: 1, Resistor_SMD:R_0805_2012Metric
- removed conn1, conn2: ~, module-custom-for-esp8266:connector-10
- added J2: Conn_01x12_Pin, module-custom-for-esp8266:connector-12-green-mini, F.Cu at (119.7, 109.8)
- added J3: Conn_01x12_Pin, module-custom-for-esp8266:connector-12-green-mini, F.Cu at (123.6, 61.7)
- added Jumper-d5: 1, Resistor_SMD:R_0805_2012Metric, B.Cu at (101.2, 78.8)
- added Jumper-d6: 1, Resistor_SMD:R_0805_2012Metric, B.Cu at (90.5, 77.0)
- added Jumper-d7: 1, Resistor_SMD:R_0805_2012Metric, B.Cu at (83.2, 77.5)
- added K3-possible-d1: ZC32F-012-HS3-copy, module-custom-for-esp8266:ZC32F-012-HS3, F.Cu at (89.3, 83.8)
- added MX-RM-5V-RF-sensor1: Conn_01x04_Pin, module-custom-for-esp8266:RF_Receiver_433_MHz, F.Cu at (79.5, 71.5)
- added U7: DS18B20, Package_TO_SOT_THT:TO-92_Inline, F.Cu at (88.0, 129.7)
- added display/ads1: Conn_01x04_Pin, Connector_PinHeader_2.54mm:PinHeader_1x04_P2.54mm_Vertical, F.Cu at (81.8, 121.2)
- added jumper-d1: 0, Resistor_SMD:R_0805_2012Metric, B.Cu at (93.0, 102.6)
- added max1: Conn_01x05_Pin, Connector_PinHeader_2.54mm:PinHeader_1x05_P2.54mm_Vertical, F.Cu at (98.3, 102.3)
- IRLR1, IRLR2, IRLR3: footprint IRLR3103:DPAK229P990X239-4N -> Package_TO_SOT_SMD:TO-252-2
- J1: value Program-connector -> Conn_01x05_Pin; footprint Connector_PinHeader_2.54mm:PinHeader_1x04_P2.54mm_Vertical -> Connector_PinHeader_2.54mm:PinHeader_1x05_P2.54mm_Vertical
- Q1, Q2, Q3, Q4, R10, R11, R12, R13, R14, R15, R16, R17, R18, U6: moved to B.Cu
- R3: value 1 -> 100; moved to F.Cu
- moved Q4 134.0 mm to (80.0, 91.7), turned to 180 degrees
- moved R14 130.8 mm to (80.9, 88.1), turned to 90 degrees
- moved D1 120.6 mm to (125.4, 128.4), turned to 180 degrees
- moved R16 119.4 mm to (102.5, 112.6), turned to 90 degrees
- moved R17 118.5 mm to (91.0, 88.6), turned to 90 degrees
- moved Q2 118.2 mm to (100.4, 92.2), turned to 180 degrees
- moved R18 107.9 mm to (101.3, 88.7), turned to 90 degrees
- moved Q3 106.9 mm to (110.8, 92.3), turned to 180 degrees
- moved R15 101.3 mm to (111.8, 88.9), turned to 90 degrees
- moved K4 99.0 mm to (99.8, 83.8), turned to 90 degrees
- moved K2 95.8 mm to (110.1, 83.8), turned to 90 degrees
- moved dc-in1 87.4 mm to (114.7, 117.7), turned to 180 degrees
- moved R10 80.1 mm to (101.8, 120.8), turned to -90 degrees
- moved Q1 76.1 mm to (90.1, 92.0), turned to 180 degrees
- moved R11 74.7 mm to (102.6, 118.0)
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Connections:
- J1 pad 4: GNDPWR -> /d3
- K1 pad 1: Net-(Q1-C) -> Net-(Q4-C)
- K2 pad 1: Net-(Q2-C) -> Net-(Q3-C)
- K4 pad 1: Net-(Q4-C) -> Net-(Q2-C)
- R14 pad 1: Net-(Q1-B) -> Net-(Q4-B)
- R15 pad 1: Net-(Q2-B) -> Net-(Q3-B)
- R17 pad 1: Net-(Q3-B) -> Net-(Q1-B)
- R18 pad 1: Net-(Q4-B) -> Net-(Q2-B)
- R3 pad 1: /d5 -> Net-(R3-Pad1)
- R3 pad 2: /mosf1-out-d5 -> /a0
- RV1 pad 2: /a0 -> Net-(R3-Pad1)
Routing:
- net GNDPWR: track 0.00 -> 342.8 mm
- net +5C: track 0.00 -> 185.4 mm
- net +3.3V: track 0.00 -> 108.0 mm, vias 0 -> 1
- net /d1: track 0.00 -> 100.1 mm, vias 0 -> 1
- net +12C: track 0.00 -> 93.5 mm
- net /d5: track 0.00 -> 90.7 mm, vias 0 -> 1
- net /d7: track 0.00 -> 87.3 mm, vias 0 -> 1
- net /conn1-10: track 0.00 -> 85.0 mm
- net /d2: track 0.00 -> 81.5 mm
- net /tx: track 0.00 -> 72.5 mm, vias 0 -> 1
- net /mosf3-out-d7: track 0.00 -> 63.7 mm
- net /a0-in-res: track 0.00 -> 63.3 mm
- net /mosf1-out-d5: track 0.00 -> 57.9 mm
- net /d8: track 0.00 -> 57.6 mm, vias 0 -> 1
- net /d3: track 0.00 -> 55.8 mm
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Other:
- board outline added: 50 x 77.2 mm
