File: IoTmanager/IoTmanager.kicad_pcb (KiCad board)
At the start: 2 copper layers, 41 parts, among them J1 Program-connector, K1 ZC32F-012-HS3-copy, K2 ZC32F-012-HS3-copy, K3 ZC32F-012-HS3-copy, K4 ZC32F-012-HS3-copy, Q1 BC817, Q2 BC817, Q3 BC817, Q4 BC817, U2 ESP-12F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

Commit message: 123
Parts:
- removed Flash1: SW_Omron_B3FS, Button_Switch_SMD:SW_SPST_Omron_B3FS-100xP
- removed K1, K2, K4: ZC32F-012-HS3-copy, module-custom-for-esp8266:ZC32F-012-HS3
- removed Q2, Q3, Q4: BC817, Package_TO_SOT_SMD:SOT-23
- removed R14, R15, R18: 1k, Resistor_SMD:R_0805_2012Metric
- removed R7: 1, Resistor_SMD:R_0805_2012Metric
- removed conn1, conn2: ~, module-custom-for-esp8266:connector-10
- added C1: C_Polarized_1000mF, Capacitor_THT:CP_Radial_D10.0mm_P3.50mm, F.Cu at (86.9, 74.8)
- added J2: Conn_01x12_Pin, module-custom-for-esp8266:connector-12-green-mini, F.Cu at (119.7, 118.5)
- added J3: Conn_01x12_Pin, module-custom-for-esp8266:connector-12-green-mini, F.Cu at (123.6, 61.7)
- added J4: flash, Connector_PinHeader_2.54mm:PinHeader_1x02_P2.54mm_Vertical, F.Cu at (113.6, 100.9)
- added J5: reset, Connector_PinHeader_2.54mm:PinHeader_1x02_P2.54mm_Vertical, F.Cu at (113.7, 104.5)
- added Jumper-d5: 1, Resistor_SMD:R_0805_2012Metric, B.Cu at (104.3, 78.3)
- added Jumper-d6: 1, Resistor_SMD:R_0805_2012Metric, B.Cu at (90.3, 78.6)
- added Jumper-d7: 1, Resistor_SMD:R_0805_2012Metric, B.Cu at (80.4, 78.2)
- added K5: ZC32F-012-HS3-copy, module-custom-for-esp8266:ZC32F-012-HS3, F.Cu at (89.5, 84.3)
- added K6: ZC32F-012-HS3-copy, module-custom-for-esp8266:ZC32F-012-HS3, F.Cu at (99.9, 84.3)
- added K7: ZC32F-012-HS3-copy, module-custom-for-esp8266:ZC32F-012-HS3, F.Cu at (110.3, 84.3)
- added MX-RM-5V-RF-sensor1: Conn_01x04_Pin, module-custom-for-esp8266:RF_Receiver_433_MHz, F.Cu at (79.7, 66.6)
- added Q10: MMBT5401, Package_TO_SOT_SMD:SOT-23, B.Cu at (113.7, 88.8)
- added Q11: MMBT5551-npn, Package_TO_SOT_SMD:SOT-23, B.Cu at (113.7, 94.2)
- added Q5: MMBT5401, Package_TO_SOT_SMD:SOT-23, B.Cu at (82.8, 88.8)
- added Q6: MMBT5551-npn, Package_TO_SOT_SMD:SOT-23, B.Cu at (82.8, 94.2)
- added Q7: MMBT5551-npn, Package_TO_SOT_SMD:SOT-23, B.Cu at (93.0, 94.1)
- added Q8: MMBT5401, Package_TO_SOT_SMD:SOT-23, B.Cu at (103.5, 88.8)
- added Q9: MMBT5551-npn, Package_TO_SOT_SMD:SOT-23, B.Cu at (103.5, 94.4)
- added R21: R-1k, Resistor_SMD:R_0805_2012Metric, B.Cu at (82.5, 86.0)
- added R22: R-1k, Resistor_SMD:R_0805_2012Metric, B.Cu at (82.5, 91.5)
- added R23: R-1k, Resistor_SMD:R_0805_2012Metric, B.Cu at (103.3, 86.1)
- added R24: R-1k, Resistor_SMD:R_0805_2012Metric, B.Cu at (103.3, 91.7)
- added R25: R-1k, Resistor_SMD:R_0805_2012Metric, B.Cu at (113.5, 86.1)
- added R26: R-1k, Resistor_SMD:R_0805_2012Metric, B.Cu at (113.5, 91.5)
- added U12: AMS1117-5.0, Package_TO_SOT_SMD:SOT-223-3_TabPin2, B.Cu at (113.2, 76.1)
- added U7: DS18B20, Package_TO_SOT_THT:TO-92_Inline, F.Cu at (111.1, 123.6)
- added display/ads1: Conn_01x04_Pin, Connector_PinHeader_2.54mm:PinHeader_1x04_P2.54mm_Vertical, F.Cu at (79.4, 115.7)
- added max1: ~, Connector_PinHeader_2.54mm:PinHeader_1x05_P2.54mm_Vertical, F.Cu at (117.3, 111.0)
- IRLR1, IRLR2, IRLR3: footprint IRLR3103:DPAK229P990X239-4N -> Package_TO_SOT_SMD:TO-252-2
- J1: value Program-connector -> prog
- Q1: value BC817 -> MMBT5401; moved to B.Cu
- R1, R5, R8: value 100 -> R-100
- R10, R11, R12, R13: value 10k -> R-10k; moved to B.Cu
- R16: value 100 -> R-100; moved to B.Cu
- R17: value 1k -> R-1k; moved to B.Cu
- R2, R6, R9: value 10k -> R-10k
- R3: value 1 -> R-100
- R4: value 1 -> R-1k
- U3: footprint OptoDevice:Vishay_MINICAST-3Pin -> OptoDevice:Vishay_MOLD-3Pin
- U4: footprint Mini360_step-down:Mini360_step-down -> module-custom-for-esp8266:Mini360_step-down
- U6: moved to B.Cu
- moved D1 146.6 mm to (88.0, 121.8), turned to 180 degrees
- moved K3 121.7 mm to (79.1, 84.3), turned to 90 degrees
- moved R17 117.7 mm to (92.8, 91.4)
- moved R16 116.2 mm to (101.8, 105.0), turned to 90 degrees
- moved U3 73.8 mm to (81.7, 118.8), turned to -90 degrees
- moved R10 73.7 mm to (101.0, 113.2), turned to -90 degrees
- moved U6 73.6 mm to (114.4, 117.1)
- moved Q1 71.6 mm to (93.0, 88.7), turned to 180 degrees
- moved R11 68.6 mm to (101.8, 110.4)
- moved R13 68.3 mm to (97.5, 104.2), turned to 90 degrees
- moved R12 68.2 mm to (98.3, 110.4)
- moved J1 65.9 mm to (88.8, 115.7), turned to 180 degrees
- moved R3 55.4 mm to (105.0, 112.9), turned to -90 degrees
- moved dc-in1 44.1 mm to (114.7, 68.3), turned to 180 degrees
- moved U2 40.1 mm to (100.1, 113.3), turned to 180 degrees
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Connections:
- J1 pad 1: +3.3V -> +5C
- J1 pad 2: /tx -> GNDPWR
- J1 pad 3: /rx -> /tx
- J1 pad 4: GNDPWR -> /rx
- Q1 pad 2: GNDPWR -> +3.3V
- R17 pad 2: /d3 -> Net-(Q1-C)
- R3 pad 1: /d5 -> Net-(R3-Pad1)
- R3 pad 2: /mosf1-out-d5 -> /a0
- R4 pad 1: /d6 -> Net-(Q1-B)
- R4 pad 2: /mosf2-out-d6 -> /tx
- RV1 pad 2: /a0 -> Net-(R3-Pad1)
Routing:
- net GNDPWR: track 0.00 -> 324.6 mm, vias 0 -> 1
- net +5C: track 0.00 -> 232.1 mm
- net /d5: track 0.00 -> 118.2 mm
- net /d7: track 0.00 -> 102.0 mm, vias 0 -> 1
- net /d1: track 0.00 -> 97.2 mm
- net +3.3V: track 0.00 -> 92.9 mm, vias 0 -> 5
- net /mosf3-out-d7: track 0.00 -> 92.4 mm
- net /mosf2-out-d6: track 0.00 -> 90.1 mm
- net /tx: track 0.00 -> 83.7 mm, vias 0 -> 2
- net /mosf1-out-d5: track 0.00 -> 77.7 mm
- net /d0: track 0.00 -> 76.9 mm, vias 0 -> 2
- net /d2: track 0.00 -> 75.2 mm, vias 0 -> 2
- net /d3: track 0.00 -> 61.2 mm, vias 0 -> 2
- net /d6: track 0.00 -> 60.2 mm
- net /conn2-1: track 0.00 -> 54.2 mm
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- added copper zone on B.Cu, net GNDPWR
- added copper zone on F.Cu, net GNDPWR
Other:
- board outline added: 50 x 70.7 mm

Commit message: update
Changed lines of the file:
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@@
 		(at 79.1 84.3 90)
 		(property "Reference" "K3"
-			(at -14.9 -1.9 90)
+			(at -2.0092 -0.4108 90)
 			(unlocked yes)
 			(layer "F.SilkS")
