File: IoTmanager/IoTmanager-v2.kicad_sch (KiCad schematic)
At the start: 58 parts, among them J1 prog, J2 Conn_01x12_Pin, J3 Conn_01x12_Pin, J4 flash, J5 reset, K3 ZC32F-012-HS3-copy, K5 ZC32F-012-HS3-copy, K6 ZC32F-012-HS3-copy, K7 ZC32F-012-HS3-copy, Q1 MMBT5401, Q10 MMBT5401, Q11 MMBT5551-npn, Q5 MMBT5401, Q6 MMBT5551-npn, Q7 MMBT5551-npn, Q8 MMBT5401, Q9 MMBT5551-npn, U1 NodeMCU_1.0_(ESP-12E), U12 AMS1117-5.0, U2 ESP-12F, U3 TSOP23xx, U4 Mini360, U5 PJ-320A, U6 AMS1117-3.3, U7 DS18B20

Commit message: update
Parts:
- K3, K5, K6: footprint module-custom-for-esp8266:ZC32F-012-HS3 -> module-custom-for-esp8266:HF32F-005-ZS3
- K7: footprint module-custom-for-esp8266:ZC32F-012-HS3 -> module-custom-for-esp8266:HF32F-005-ZS3; symbol models:ZC32F-012-HS3-copy -> models:ZC32F-012-HS3
- renumbered J4 to J4-flash1, Q1 to Q1-pnp1, Q10 to Q10-pnp1, Q11 to Q11-npn1, Q7 to Q7-npn1, Q8 to Q8-pnp1, R10 to R10-10k1, R11 to R11-10k1, R12 to R12-10k1, U3 to U3-tsop23, J1 to prog1
Changed lines of the file:
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@@
 		(on_board yes)
 		(dnp no)
-		(property "Reference" "R10"
+		(property "Reference" "R10-10k1"
 			(at 96.52 155.448 90)
 			(effects
@@
 			(project "IoTmanager"
 				(path "/e30adb8f-2050-4707-a23b-b56498f87e6f"
-					(reference "R10")
+					(reference "R10-10k1")
 					(unit 1)
 				)
@@
 	)
 	(symbol
-		(lib_id "models:ZC32F-012-HS3-copy")
+		(lib_id "models:ZC32F-012-HS3")
 		(at 270.51 248.92 0)
 		(unit 1)
@@
 		)
 		(property "Value" "ZC32F-012-HS3-copy"
-			(at 281.94 250.1899 0)
+			(at 281.94 248.9199 0)
 			(effects
 				(font
@@
 			)
 		)
-		(property "Footprint" "module-custom-for-esp8266:ZC32F-012-HS3"
+		(property "Footprint" "module-custom-for-esp8266:HF32F-005-ZS3"
 			(at 281.94 250.19 0)
 			(effects
@@
 			)
 		)
-		(property "Footprint" "module-custom-for-esp8266:ZC32F-012-HS3"
+		(property "Footprint" "module-custom-for-esp8266:HF32F-005-ZS3"
 			(at 142.24 242.57 0)
 			(effects
@@
 		(on_board yes)
 		(dnp no)
-		(property "Reference" "J1"
+		(property "Reference" "prog1"
 			(at 70.485 161.29 0)
 			(effects
@@
 			(project ""
 				(path "/e30adb8f-2050-4707-a23b-b56498f87e6f"
-					(reference "J1")
+					(reference "prog1")
 					(unit 1)
 				)
@@
 		(dnp no)
 		(fields_autoplaced yes)
-		(property "Reference" "U3"
+		(property "Reference" "U3-tsop23"
 			(at 217.975 116.84 0)
 			(effects
@@
 			(project ""
 				(path "/e30adb8f-2050-4707-a23b-b56498f87e6f"
-					(reference "U3")
+					(reference "U3-tsop23")
 					(unit 1)
 				)
@@
 		(on_board yes)
 		(dnp no)
-		(property "Reference" "R12"
+		(property "Reference" "R12-10k1"
 			(at 156.21 155.448 90)
 			(effects
@@
 			(project "IoTmanager"
 				(path "/e30adb8f-2050-4707-a23b-b56498f87e6f"
-					(reference "R12")
+					(reference "R12-10k1")
 					(unit 1)
 				)
@@
 			)
 		)
-		(property "Footprint" "module-custom-for-esp8266:ZC32F-012-HS3"
+		(property "Footprint" "module-custom-for-esp8266:HF32F-005-ZS3"
 			(at 64.77 238.76 0)
 			(effects
@@
 		(dnp no)
 		(fields_autoplaced yes)
-		(property "Reference" "Q11"
+		(property "Reference" "Q11-npn1"
 			(at 267.97 260.3499 0)
 			(effects
@@
 			(project "IoTmanager"
 				(path "/e30adb8f-2050-4707-a23b-b56498f87e6f"
-					(reference "Q11")
+					(reference "Q11-npn1")
 					(unit 1)
 				)
@@
 		(on_board yes)
 		(dnp no)
-		(property "Reference" "R11"
+		(property "Reference" "R11-10k1"
 			(at 96.52 161.798 90)
 			(effects
@@
 			(project "IoTmanager"
 				(path "/e30adb8f-2050-4707-a23b-b56498f87e6f"
-					(reference "R11")
+					(reference "R11-10k1")
 					(unit 1)
 				)
@@
 		(dnp no)
 		(fields_autoplaced yes)
-		(property "Reference" "Q10"
+		(property "Reference" "Q10-pnp1"
 			(at 247.65 273.0499 0)
 			(effects
@@
 			(project "IoTmanager"
 				(path "/e30adb8f-2050-4707-a23b-b56498f87e6f"
-					(reference "Q10")
+					(reference "Q10-pnp1")
 					(unit 1)
 				)
@@
 		(dnp no)
 		(fields_autoplaced yes)
-		(property "Reference" "J4"
+		(property "Reference" "J4-flash1"
 			(at 85.725 181.61 0)
 			(effects
@@
 			(project ""
 				(path "/e30adb8f-2050-4707-a23b-b56498f87e6f"
-					(reference "J4")
+					(reference "J4-flash1")
 					(unit 1)
 				)
@@
 		(dnp no)
 		(fields_autoplaced yes)
-		(property "Reference" "Q7"
+		(property "Reference" "Q7-npn1"
 			(at 128.27 252.7299 0)
 			(effects
@@
 			(project "IoTmanager"
 				(path "/e30adb8f-2050-4707-a23b-b56498f87e6f"
-					(reference "Q7")
+					(reference "Q7-npn1")
 					(unit 1)
 				)
@@
 			)
 		)
-		(property "Footprint" "module-custom-for-esp8266:ZC32F-012-HS3"
+		(property "Footprint" "module-custom-for-esp8266:HF32F-005-ZS3"
 			(at 209.55 246.38 0)
 			(effects
@@
 		(dnp no)
 		(fields_autoplaced yes)
-		(property "Reference" "Q1"
+		(property "Reference" "Q1-pnp1"
 			(at 107.95 265.4299 0)
 			(effects
@@
 			(project "IoTmanager"
 				(path "/e30adb8f-2050-4707-a23b-b56498f87e6f"
-					(reference "Q1")
+					(reference "Q1-pnp1")
 					(unit 1)
 				)
@@
 		(dnp no)
 		(fields_autoplaced yes)
-		(property "Reference" "Q8"
+		(property "Reference" "Q8-pnp1"
 			(at 175.26 269.2399 0)
 			(effects
@@
 			(project "IoTmanager"
 				(path "/e30adb8f-2050-4707-a23b-b56498f87e6f"
-					(reference "Q8")
+					(reference "Q8-pnp1")
 					(unit 1)
 				)

Commit message: update
Parts:
- added D2, D3, D4, D5: 1N4148, module-custom-for-esp8266:sod80-1n1448, symbol models:1N4148
Connections:
- net +5C: now also D2.1 (K), D3.1 (K), D4.1 (K), D5.1 (K)
- net at K6.1, Q9.3 (C): now also D4.2 (A)
- net at K7.1, Q11-npn1.3 (C): now also D5.2 (A)
- net at K5.1, Q7-npn1.3 (C): now also D3.2 (A)
- net at K3.1, Q6.3 (C): now also D2.2 (A)

Commit message: update
Parts:
- added R7: R-4k7, Resistor_SMD:R_0805_2012Metric, symbol models:R-1k
Connections:
- net +5C: now also R7.2
- net d3: now also U7.2 (DQ), R7.1
- net d7: no longer U7.2 (DQ)
Changed lines of the file:
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@@
 	)
 	(junction
+		(at 45.72 22.86)
+		(diameter 0)
+		(color 0 0 0 0)
+	)
+	(junction
 		(at 270.51 62.23)
 		(diameter 0)
@@
 	(wire
 		(pts
+			(xy 57.15 34.29) (xy 57.15 36.83)
+		)
+		(stroke
+			(width 0)
+			(type default)
+		)
+	)
+	(wire
+		(pts
 			(xy 172.72 257.81) (xy 173.99 257.81)
 		)
@@
 	(wire
 		(pts
+			(xy 57.15 26.67) (xy 57.15 22.86)
+		)
+		(stroke
+			(width 0)
+			(type default)
+		)
+	)
+	(wire
+		(pts
 			(xy 29.21 100.33) (xy 41.91 100.33)
 		)
@@
 	(wire
 		(pts
+			(xy 45.72 22.86) (xy 45.72 29.21)
+		)
+		(stroke
+			(width 0)
+			(type default)
+		)
+	)
+	(wire
+		(pts
 			(xy 181.61 257.81) (xy 185.42 257.81)
 		)
@@
 	(wire
 		(pts
+			(xy 45.72 21.59) (xy 45.72 22.86)
+		)
+		(stroke
+			(width 0)
+			(type default)
+		)
+	)
+	(wire
+		(pts
 			(xy 165.1 111.76) (xy 168.91 111.76)
 		)
@@
 	(wire
 		(pts
+			(xy 45.72 22.86) (xy 57.15 22.86)
+		)
+		(stroke
+			(width 0)
+			(type default)
+		)
+	)
+	(wire
+		(pts
 			(xy 275.59 256.54) (xy 275.59 259.08)
 		)
@@
 		)
 	)
+	(wire
+		(pts
+			(xy 57.15 36.83) (xy 53.34 36.83)
+		)
+		(stroke
+			(width 0)
+			(type default)
+		)
+	)
 	(label "d2"
 		(at 140.97 167.64 0)
@@
 		)
 	)
-	(label "d7"
+	(label "d3"
 		(at 53.34 36.83 0)
 		(fields_autoplaced yes)
@@
 	(symbol
 		(lib_id "power:+5C")
-		(at 45.72 29.21 0)
+		(at 45.72 21.59 0)
 		(unit 1)
 		(exclude_from_sim no)
@@
 		(fields_autoplaced yes)
 		(property "Reference" "#PWR038"
-			(at 45.72 33.02 0)
+			(at 45.72 25.4 0)
 			(effects
 				(font
@@
 		)
 		(property "Value" "+5C"
-			(at 45.72 24.13 0)
+			(at 45.72 16.51 0)
 			(effects
 				(font
@@
 		)
 		(property "Footprint" ""
-			(at 45.72 29.21 0)
+			(at 45.72 21.59 0)
 			(effects
 				(font
@@
 		)
 		(property "Datasheet" ""
-			(at 45.72 29.21 0)
+			(at 45.72 21.59 0)
 			(effects
 				(font
@@
 		)
 		(property "Description" "Power symbol creates a global label with name \"+5C\""
-			(at 45.72 29.21 0)
+			(at 45.72 21.59 0)
 			(effects
 				(font
@@
 					(unit 1)
 				)
+			)
+		)
+	)
+	(symbol
+		(lib_id "models:R-1k")
+		(at 57.15 30.48 180)
+		(unit 1)
+		(exclude_from_sim no)
+		(in_bom yes)
+		(on_board yes)
+		(dnp no)
+		(fields_autoplaced yes)
+		(property "Reference" "R7"
+			(at 59.69 27.9399 0)
+			(effects
+				(font
+					(size 1.27 1.27)
+				)
+				(justify right)
+			)
+		)
+		(property "Value" "R-4k7"
+			(at 59.69 30.4799 0)
+			(effects
+				(font
+					(size 1.27 1.27)
+				)
+				(justify right)
+			)
+		)
+		(property "Footprint" "Resistor_SMD:R_0805_2012Metric"
+			(at 58.928 30.48 90)
+			(effects
+				(font
+					(size 1.27 1.27)
+				)
+				(hide yes)
+			)
+		)
+		(property "Datasheet" "~"
+			(at 57.15 30.48 0)
+			(effects
+				(font
+					(size 1.27 1.27)
+				)
+				(hide yes)
+			)
+		)
+		(property "Description" "Resistor"
+			(at 57.15 30.48 0)
+			(effects
+				(font
+					(size 1.27 1.27)
+				)
+				(hide yes)
+			)
+		)
+		(property "JLCPCB Part" "C25905"
+			(at 59.69 33.0199 0)
+			(effects
+				(font
+					(size 1.27 1.27)
+				)
+				(justify right)
+			)
+		)
+		(pin "2"
+		)
+		(pin "1"
+		)
+		(instances
+			(project ""
+				(path "/e30adb8f-2050-4707-a23b-b56498f87e6f"
+					(reference "R7")
+					(unit 1)
+				)

Commit message: update
Connections:
- net d2: now also R7.1, U7.2 (DQ)
- net d3: no longer R7.1, U7.2 (DQ)
Changed lines of the file:
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@@
 		)
 	)
-	(label "d3"
+	(label "d2"
 		(at 53.34 36.83 0)
 		(fields_autoplaced yes)

Commit message: update
Connections:
- net +3.3V: now also C1.1
- net +5C: no longer C1.1
Other:
- moved on the sheet: C1
Changed lines of the file:
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@@
 	)
 	(junction
-		(at 29.21 100.33)
-		(diameter 0)
-		(color 0 0 0 0)
-	)
-	(junction
 		(at 261.62 72.39)
 		(diameter 0)
@@
 	)
 	(junction
-		(at 36.83 88.9)
+		(at 102.87 157.48)
 		(diameter 0)
 		(color 0 0 0 0)
 	)
 	(junction
-		(at 102.87 157.48)
+		(at 87.63 138.43)
 		(diameter 0)
 		(color 0 0 0 0)
@@
 	)
 	(junction
+		(at 99.06 128.27)
+		(diameter 0)
+		(color 0 0 0 0)
+	)
+	(junction
 		(at 147.32 157.48)
 		(diameter 0)
@@
 	(wire
 		(pts
-			(xy 41.91 88.9) (xy 36.83 88.9)
-		)
-		(stroke
-			(width 0)
-			(type default)
-		)
-	)
-	(wire
-		(pts
 			(xy 115.57 248.92) (xy 125.73 248.92)
 		)
@@
 	(wire
 		(pts
+			(xy 99.06 128.27) (xy 99.06 130.81)
+		)
+		(stroke
+			(width 0)
+			(type default)
+		)
+	)
+	(wire
+		(pts
 			(xy 148.59 73.66) (xy 158.75 73.66)
 		)
@@
 	(wire
 		(pts
-			(xy 29.21 96.52) (xy 29.21 100.33)
+			(xy 158.75 63.5) (xy 161.29 63.5)
 		)
 		(stroke
@@
 	(wire
 		(pts
-			(xy 158.75 63.5) (xy 161.29 63.5)
+			(xy 250.19 72.39) (xy 250.19 62.23)
 		)
 		(stroke
@@
 	(wire
 		(pts
-			(xy 250.19 72.39) (xy 250.19 62.23)
+			(xy 215.9 73.66) (xy 215.9 83.82)
 		)
 		(stroke
@@
 	(wire
 		(pts
-			(xy 215.9 73.66) (xy 215.9 83.82)
+			(xy 99.06 128.27) (xy 104.14 128.27)
 		)
 		(stroke
@@
 	(wire
 		(pts
-			(xy 29.21 100.33) (xy 41.91 100.33)
-		)
-		(stroke
-			(width 0)
-			(type default)
-		)
-	)
-	(wire
-		(pts
 			(xy 170.18 73.66) (xy 171.45 73.66)
 		)
@@
 	(wire
 		(pts
-			(xy 172.72 265.43) (xy 172.72 257.81)
+			(xy 99.06 135.89) (xy 99.06 138.43)
 		)
 		(stroke
@@
 	(wire
 		(pts
-			(xy 134.62 97.79) (xy 139.7 97.79)
+			(xy 172.72 265.43) (xy 172.72 257.81)
 		)
 		(stroke
@@
 	(wire
 		(pts
-			(xy 74.93 171.45) (xy 77.47 171.45)
+			(xy 134.62 97.79) (xy 139.7 97.79)
 		)
 		(stroke
@@
 	(wire
 		(pts
-			(xy 41.91 95.25) (xy 41.91 88.9)
+			(xy 74.93 171.45) (xy 77.47 171.45)
 		)
 		(stroke
@@
 	(wire
 		(pts
-			(xy 95.25 128.27) (xy 104.14 128.27)
+			(xy 95.25 128.27) (xy 99.06 128.27)
 		)
 		(stroke
@@
 	(wire
 		(pts
+			(xy 87.63 138.43) (xy 87.63 139.7)
+		)
+		(stroke
+			(width 0)
+			(type default)
+		)
+	)
+	(wire
+		(pts
 			(xy 165.1 111.76) (xy 168.91 111.76)
 		)
@@
 	(wire
 		(pts
-			(xy 87.63 135.89) (xy 87.63 139.7)
+			(xy 87.63 135.89) (xy 87.63 138.43)
+		)
+		(stroke
+			(width 0)
+			(type default)
+		)
+	)
+	(wire
+		(pts
+			(xy 99.06 138.43) (xy 87.63 138.43)
 		)
 		(stroke
@@
 	(wire
 		(pts
-			(xy 29.21 100.33) (xy 29.21 101.6)
+			(xy 29.21 96.52) (xy 29.21 101.6)
 		)
 		(stroke
@@
 	(symbol
 		(lib_id "resistor:C_Polarized_Small")
-		(at 41.91 97.79 0)
+		(at 99.06 133.35 0)
 		(unit 1)
 		(exclude_from_sim no)
@@
 		(fields_autoplaced yes)
 		(property "Reference" "C1"
-			(at 44.45 95.9738 0)
+			(at 101.6 131.5338 0)
 			(effects
 				(font
@@
 		)
 		(property "Value" "C_Polarized_1000mF"
-			(at 44.45 98.5138 0)
+			(at 101.6 134.0738 0)
 			(effects
 				(font
@@
 		)
 		(property "Footprint" "Capacitor_THT:CP_Radial_D10.0mm_P3.50mm"
-			(at 41.91 97.79 0)
+			(at 99.06 133.35 0)
 			(effects
 				(font
@@
 		)
 		(property "Datasheet" "~"
-			(at 41.91 97.79 0)
+			(at 99.06 133.35 0)
 			(effects
 				(font
@@
 		)
 		(property "Description" "Polarized capacitor, small symbol"
-			(at 41.91 97.79 0)
+			(at 99.06 133.35 0)
 			(effects
 				(font
@@
 		)
 		(property "Supplier" ""
-			(at 41.91 97.79 0)
+			(at 99.06 133.35 0)
 			(effects
 				(font

Commit message: update
Parts:
- U7: footprint Package_TO_SOT_THT:TO-92_Inline -> Connector_PinHeader_2.54mm:PinHeader_1x03_P2.54mm_Vertical
Changed lines of the file:
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@@
 	(wire
 		(pts
+			(xy 193.04 228.6) (xy 193.04 237.49)
+		)
+		(stroke
+			(width 0)
+			(type default)
+		)
+	)
+	(wire
+		(pts
 			(xy 260.35 72.39) (xy 261.62 72.39)
 		)
@@
 	(wire
 		(pts
-			(xy 48.26 223.52) (xy 48.26 227.33)
+			(xy 48.26 219.71) (xy 48.26 227.33)
 		)
 		(stroke
@@
 	(wire
 		(pts
-			(xy 125.73 227.33) (xy 125.73 232.41)
+			(xy 125.73 222.25) (xy 125.73 232.41)
 		)
 		(stroke
@@
 	(wire
 		(pts
+			(xy 265.43 231.14) (xy 265.43 241.3)
+		)
+		(stroke
+			(width 0)
+			(type default)
+		)
+	)
+	(wire
+		(pts
 			(xy 140.97 160.02) (xy 138.43 160.02)
 		)
@@
 	(symbol
 		(lib_id "power:+12C")
-		(at 125.73 227.33 0)
+		(at 125.73 222.25 0)
 		(unit 1)
 		(exclude_from_sim no)
@@
 		(fields_autoplaced yes)
 		(property "Reference" "#PWR034"
-			(at 125.73 231.14 0)
+			(at 125.73 226.06 0)
 			(effects
 				(font
@@
 		)
 		(property "Value" "+5C"
-			(at 125.73 222.25 0)
+			(at 125.73 217.17 0)
 			(effects
 				(font
@@
 		)
 		(property "Footprint" ""
-			(at 125.73 227.33 0)
+			(at 125.73 222.25 0)
 			(effects
 				(font
@@
 		)
 		(property "Datasheet" ""
-			(at 125.73 227.33 0)
+			(at 125.73 222.25 0)
 			(effects
 				(font
@@
 		)
 		(property "Description" "Power symbol creates a global label with name \"+12C\""
-			(at 125.73 227.33 0)
+			(at 125.73 222.25 0)
 			(effects
 				(font
@@
 	(symbol
 		(lib_id "power:+12C")
-		(at 48.26 223.52 0)
+		(at 48.26 219.71 0)
 		(unit 1)
 		(exclude_from_sim no)
@@
 		(fields_autoplaced yes)
 		(property "Reference" "#PWR047"
-			(at 48.26 227.33 0)
+			(at 48.26 223.52 0)
 			(effects
 				(font
@@
 		)
 		(property "Value" "+5C"
-			(at 48.26 218.44 0)
+			(at 48.26 214.63 0)
 			(effects
 				(font
@@
 		)
 		(property "Footprint" ""
-			(at 48.26 223.52 0)
+			(at 48.26 219.71 0)
 			(effects
 				(font
@@
 		)
 		(property "Datasheet" ""
-			(at 48.26 223.52 0)
+			(at 48.26 219.71 0)
 			(effects
 				(font
@@
 		)
 		(property "Description" "Power symbol creates a global label with name \"+12C\""
-			(at 48.26 223.52 0)
+			(at 48.26 219.71 0)
 			(effects
 				(font
@@
 			)
 		)
-		(property "Footprint" "Package_TO_SOT_THT:TO-92_Inline"
+		(property "Footprint" "Connector_PinHeader_2.54mm:PinHeader_1x03_P2.54mm_Vertical"
 			(at 20.32 43.18 0)
 			(effects
@@
 	(symbol
 		(lib_id "power:+12C")
-		(at 193.04 237.49 0)
+		(at 193.04 228.6 0)
 		(unit 1)
 		(exclude_from_sim no)
@@
 		(fields_autoplaced yes)
 		(property "Reference" "#PWR051"
-			(at 193.04 241.3 0)
+			(at 193.04 232.41 0)
 			(effects
 				(font
@@
 		)
 		(property "Value" "+5C"
-			(at 193.04 232.41 0)
+			(at 193.04 223.52 0)
 			(effects
 				(font
@@
 		)
 		(property "Footprint" ""
-			(at 193.04 237.49 0)
+			(at 193.04 228.6 0)
 			(effects
 				(font
@@
 		)
 		(property "Datasheet" ""
-			(at 193.04 237.49 0)
+			(at 193.04 228.6 0)
 			(effects
 				(font
@@
 		)
 		(property "Description" "Power symbol creates a global label with name \"+12C\""
-			(at 193.04 237.49 0)
+			(at 193.04 228.6 0)
 			(effects
 				(font
@@
 	(symbol
 		(lib_id "power:+12C")
-		(at 265.43 241.3 0)
+		(at 265.43 231.14 0)
 		(unit 1)
 		(exclude_from_sim no)
@@
 		(fields_autoplaced yes)
 		(property "Reference" "#PWR054"
-			(at 265.43 245.11 0)
+			(at 265.43 234.95 0)
 			(effects
 				(font
@@
 		)
 		(property "Value" "+5C"
-			(at 265.43 236.22 0)
+			(at 265.43 226.06 0)
 			(effects
 				(font
@@
 		)
 		(property "Footprint" ""
-			(at 265.43 241.3 0)
+			(at 265.43 231.14 0)
 			(effects
 				(font
@@
 		)
 		(property "Datasheet" ""
-			(at 265.43 241.3 0)
+			(at 265.43 231.14 0)
 			(effects
 				(font
@@
 		)
 		(property "Description" "Power symbol creates a global label with name \"+12C\""
-			(at 265.43 241.3 0)
+			(at 265.43 231.14 0)
 			(effects
 				(font

Commit message: update
Connections:
- net +12C: now also J2.12 (Pin_12)
- net GNDPWR: no longer J3.12 (Pin_12)
- net conn1-10: now also J3.12 (Pin_12); no longer J2.11 (Pin_11)
- net conn1-8: now also J3.10 (Pin_10); no longer J2.9 (Pin_9)
- net conn1-9: now also J3.11 (Pin_11); no longer J2.10 (Pin_10)
- net d0: now also J2.9 (Pin_9); no longer J3.11 (Pin_11)
- net d1: now also J2.10 (Pin_10); no longer J2.12 (Pin_12)
- net d2: now also J2.11 (Pin_11); no longer J3.10 (Pin_10)
Changed lines of the file:
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@@
 	(wire
 		(pts
+			(xy 265.43 167.64) (xy 264.16 167.64)
+		)
+		(stroke
+			(width 0)
+			(type default)
+		)
+	)
+	(wire
+		(pts
 			(xy 138.43 180.34) (xy 153.67 180.34)
 		)
@@
 	(wire
 		(pts
+			(xy 260.35 218.44) (xy 265.43 218.44)
+		)
+		(stroke
+			(width 0)
+			(type default)
+		)
+	)
+	(wire
+		(pts
 			(xy 260.35 190.5) (xy 265.43 190.5)
 		)
@@
 	(wire
 		(pts
+			(xy 264.16 172.72) (xy 269.24 172.72)
+		)
+		(stroke
+			(width 0)
+			(type default)
+		)
+	)
+	(wire
+		(pts
 			(xy 26.67 147.32) (xy 35.56 147.32)
 		)
@@
 	(wire
 		(pts
+			(xy 264.16 177.8) (xy 269.24 177.8)
+		)
+		(stroke
+			(width 0)
+			(type default)
+		)
+	)
+	(wire
+		(pts
 			(xy 81.28 168.91) (xy 74.93 168.91)
 		)
@@
 	(wire
 		(pts
+			(xy 264.16 170.18) (xy 269.24 170.18)
+		)
+		(stroke
+			(width 0)
+			(type default)
+		)
+	)
+	(wire
+		(pts
 			(xy 104.14 167.64) (xy 107.95 167.64)
 		)
@@
 	(wire
 		(pts
+			(xy 264.16 175.26) (xy 269.24 175.26)
+		)
+		(stroke
+			(width 0)
+			(type default)
+		)
+	)
+	(wire
+		(pts
 			(xy 57.15 36.83) (xy 53.34 36.83)
 		)
@@
 	)
 	(label "conn1-9"
-		(at 264.16 172.72 0)
+		(at 265.43 215.9 0)
 		(fields_autoplaced yes)
 		(effects
@@
 	)
 	(label "d1"
-		(at 264.16 177.8 0)
+		(at 269.24 172.72 0)
 		(fields_autoplaced yes)
 		(effects
@@
 	)
 	(label "mosf3-out-d7"
-		(at 264.16 167.64 0)
+		(at 265.43 167.64 0)
 		(fields_autoplaced yes)
 		(effects
@@
 		)
 	)
-	(label "d2"
-		(at 265.43 213.36 0)
-		(fields_autoplaced yes)
-		(effects
-			(font
-				(size 1.27 1.27)
-			)
-			(justify left bottom)
-		)
-	)
 	(label "d1"
 		(at 134.62 67.31 0)
@@
 		)
 	)
-	(label "d0"
-		(at 265.43 215.9 0)
-		(fields_autoplaced yes)
-		(effects
-			(font
-				(size 1.27 1.27)
-			)
-			(justify left bottom)
-		)
-	)
 	(label "d8"
 		(at 196.85 128.27 0)
@@
 		)
 	)
+	(label "d0"
+		(at 269.24 170.18 0)
+		(fields_autoplaced yes)
+		(effects
+			(font
+				(size 1.27 1.27)
+			)
+			(justify left bottom)
+		)
+	)
 	(label "conn1-8"
-		(at 264.16 170.18 0)
+		(at 265.43 213.36 0)
 		(fields_autoplaced yes)
 		(effects
@@
 	)
 	(label "conn1-10"
-		(at 264.16 175.26 0)
+		(at 265.43 218.44 0)
 		(fields_autoplaced yes)
 		(effects
@@
 		)
 	)
+	(label "d2"
+		(at 269.24 175.26 0)
+		(fields_autoplaced yes)
+		(effects
+			(font
+				(size 1.27 1.27)
+			)
+			(justify left bottom)
+		)
+	)
 	(label "d7"
 		(at 140.97 175.26 0)
@@
 	)
 	(symbol
+		(lib_id "power:+12C")
+		(at 269.24 177.8 270)
+		(unit 1)
+		(exclude_from_sim no)
+		(in_bom yes)
+		(on_board yes)
+		(dnp no)
+		(fields_autoplaced yes)
+		(property "Reference" "#PWR033"
+			(at 265.43 177.8 0)
+			(effects
+				(font
+					(size 1.27 1.27)
+				)
+				(hide yes)
+			)
+		)
+		(property "Value" "+12C"
+			(at 273.05 177.7999 90)
+			(effects
+				(font
+					(size 1.27 1.27)
+				)
+				(justify left)
+			)
+		)
+		(property "Footprint" ""
+			(at 269.24 177.8 0)
+			(effects
+				(font
+					(size 1.27 1.27)
+				)
+				(hide yes)
+			)
+		)
+		(property "Datasheet" ""
+			(at 269.24 177.8 0)
+			(effects
+				(font
+					(size 1.27 1.27)
+				)
+				(hide yes)
+			)
+		)
+		(property "Description" "Power symbol creates a global label with name \"+12C\""
+			(at 269.24 177.8 0)
+			(effects
+				(font
+					(size 1.27 1.27)
+				)
+				(hide yes)
+			)
+		)
+		(pin "1"
+		)
+		(instances
+			(project "IoTmanager-v2"
+				(path "/e30adb8f-2050-4707-a23b-b56498f87e6f"
+					(reference "#PWR033")
+					(unit 1)
+				)
+			)
+		)
+	)
+	(symbol
 		(lib_id "power:+5C")
 		(at 168.91 109.22 270)
@@
 					(unit 1)
 				)
-			)
-		)
-	)
-	(symbol
-		(lib_id "power:GNDPWR")
-		(at 260.35 218.44 90)
-		(unit 1)
-		(exclude_from_sim no)
-		(in_bom yes)
-		(on_board yes)
-		(dnp no)
-		(fields_autoplaced yes)
-		(property "Reference" "#PWR046"
-			(at 265.43 218.44 0)
-			(effects
-				(font
-					(size 1.27 1.27)
-				)
-				(hide yes)
-			)
-		)
-		(property "Value" "GNDPWR"
-			(at 264.16 218.5669 90)
-			(effects
-				(font
-					(size 1.27 1.27)
-				)
-				(justify right)
-			)
-		)
-		(property "Footprint" ""
-			(at 261.62 218.44 0)
-			(effects
-				(font
-					(size 1.27 1.27)
-				)
-				(hide yes)
-			)
-		)
-		(property "Datasheet" ""
-			(at 261.62 218.44 0)
-			(effects
-				(font
-					(size 1.27 1.27)
-				)
-				(hide yes)
-			)
-		)
-		(property "Description" "Power symbol creates a global label with name \"GNDPWR\" , global ground"
-			(at 260.35 218.44 0)
-			(effects
-				(font
-					(size 1.27 1.27)
-				)
-				(hide yes)
-			)
-		)
-		(pin "1"
-		)
-		(instances
-			(project ""
-				(path "/e30adb8f-2050-4707-a23b-b56498f87e6f"
-					(reference "#PWR046")
-					(unit 1)
-				)

Commit message: update
Connections:
- net d2: no longer R7.1, U7.2 (DQ)
- net d4: now also R7.1, U7.2 (DQ); no longer R25.2
- net rx: now also R25.2; no longer J2.3 (Pin_3)
- net tx: no longer J2.4 (Pin_4)
Changed lines of the file:
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@@
 		)
 	)
-	(label "d2"
+	(label "d4"
 		(at 53.34 36.83 0)
 		(fields_autoplaced yes)
@@
 		)
 	)
-	(label "rx"
-		(at 264.16 154.94 0)
-		(fields_autoplaced yes)
-		(effects
-			(font
-				(size 1.27 1.27)
-			)
-			(justify left bottom)
-		)
-	)
 	(label "conn2-8"
 		(at 265.43 208.28 0)
@@
 		)
 	)
-	(label "tx"
-		(at 264.16 157.48 0)
-		(fields_autoplaced yes)
-		(effects
-			(font
-				(size 1.27 1.27)
-			)
-			(justify left bottom)
-		)
-	)
 	(label "conn2-1"
 		(at 265.43 190.5 0)
@@
 		)
 	)
-	(label "d4"
+	(label "rx"
 		(at 219.71 274.32 0)
 		(fields_autoplaced yes)
