File: IoTmanager/IoTmanager-v2.kicad_sch (KiCad schematic)
At the start: 63 parts, among them J2 Conn_01x12_Pin, J3 Conn_01x12_Pin, J4-flash1 flash, J5 reset, K3 ZC32F-012-HS3-copy, K5 ZC32F-012-HS3-copy, K6 ZC32F-012-HS3-copy, K7 ZC32F-012-HS3-copy, U1 NodeMCU_1.0_(ESP-12E), U10 MMDT4413-7-F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

Commit message: update
Parts:
- added SW1: SW_PUSH_6mm_H4.3mm, module-custom-for-esp8266:SW_PUSH_6mm_H4.3mm, symbol models:SW_PUSH_6mm_H4.3mm
Connections:
- net GNDPWR: now also SW1.2 (D)
- net at R12-10k2.1, U2.19 (GPIO4): now also SW1.1 (C)
Changed lines of the file:
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@@
 	)
 	(junction
+		(at 163.83 180.34)
+		(diameter 0)
+		(color 0 0 0 0)
+	)
+	(junction
 		(at 182.88 252.73)
 		(diameter 0)
@@
 	)
 	(junction
+		(at 142.24 167.64)
+		(diameter 0)
+		(color 0 0 0 0)
+	)
+	(junction
 		(at 265.43 241.3)
 		(diameter 0)
@@
 	(wire
 		(pts
+			(xy 142.24 162.56) (xy 142.24 167.64)
+		)
+		(stroke
+			(width 0)
+			(type default)
+		)
+	)
+	(wire
+		(pts
 			(xy 265.43 241.3) (xy 265.43 245.11)
 		)
@@
 	(wire
 		(pts
-			(xy 138.43 167.64) (xy 144.78 167.64)
+			(xy 138.43 167.64) (xy 142.24 167.64)
 		)
 		(stroke
@@
 	(wire
 		(pts
+			(xy 142.24 162.56) (xy 166.37 162.56)
+		)
+		(stroke
+			(width 0)
+			(type default)
+		)
+	)
+	(wire
+		(pts
 			(xy 123.19 190.5) (xy 123.19 193.04)
 		)
@@
 	(wire
 		(pts
+			(xy 142.24 167.64) (xy 144.78 167.64)
+		)
+		(stroke
+			(width 0)
+			(type default)
+		)
+	)
+	(wire
+		(pts
 			(xy 179.07 83.82) (xy 179.07 78.74)
 		)
@@
 	(wire
 		(pts
+			(xy 176.53 162.56) (xy 176.53 180.34)
+		)
+		(stroke
+			(width 0)
+			(type default)
+		)
+	)
+	(wire
+		(pts
 			(xy 99.06 138.43) (xy 87.63 138.43)
 		)
@@
 	(wire
 		(pts
+			(xy 176.53 180.34) (xy 163.83 180.34)
+		)
+		(stroke
+			(width 0)
+			(type default)
+		)
+	)
+	(wire
+		(pts
 			(xy 29.21 96.52) (xy 29.21 101.6)
 		)
@@
 					(unit 1)
 				)
+			)
+		)
+	)
+	(symbol
+		(lib_id "models:SW_PUSH_6mm_H4.3mm")
+		(at 171.45 162.56 0)
+		(unit 1)
+		(exclude_from_sim no)
+		(in_bom yes)
+		(on_board yes)
+		(dnp no)
+		(fields_autoplaced yes)
+		(property "Reference" "SW1"
+			(at 171.45 154.94 0)
+			(effects
+				(font
+					(size 1.27 1.27)
+				)
+			)
+		)
+		(property "Value" "SW_PUSH_6mm_H4.3mm"
+			(at 171.45 157.48 0)
+			(effects
+				(font
+					(size 1.27 1.27)
+				)
+			)
+		)
+		(property "Footprint" "module-custom-for-esp8266:SW_PUSH_6mm_H4.3mm"
+			(at 171.45 153.67 0)
+			(effects
+				(font
+					(size 1.27 1.27)
+				)
+				(hide yes)
+			)
+		)
+		(property "Datasheet" "~"
+			(at 171.45 157.48 0)
+			(effects
+				(font
+					(size 1.27 1.27)
+				)
+				(hide yes)
+			)
+		)
+		(property "Description" "Push button switch, generic, separate symbols, four pins"
+			(at 171.45 168.91 0)
+			(effects
+				(font
+					(size 1.27 1.27)
+				)
+				(hide yes)
+			)
+		)
+		(pin "2"
+		)
+		(pin "1"
+		)
+		(instances
+			(project ""
+				(path "/e30adb8f-2050-4707-a23b-b56498f87e6f"
+					(reference "SW1")
+					(unit 1)
+				)

Commit message: update
Parts:
- added R12-10k4, R12-10k5: R-1k, Resistor_SMD:R_0805_2012Metric, symbol models:R-10k
- R12-10k2, R12-10k3: value R-1k -> R-4k7
Connections:
- net d8: now also R12-10k4.2; no longer J2.12 (Pin_12)
- net tx: now also R12-10k5.2
- net at J2.9 (Pin_9): now also R12-10k5.1
- new net: J2.12 (Pin_12), R12-10k4.1
Changed lines of the file:
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@@
 	(wire
 		(pts
+			(xy 281.94 177.8) (xy 284.48 177.8)
+		)
+		(stroke
+			(width 0)
+			(type default)
+		)
+	)
+	(wire
+		(pts
 			(xy 267.97 59.69) (xy 267.97 72.39)
 		)
@@
 	(wire
 		(pts
-			(xy 264.16 177.8) (xy 269.24 177.8)
+			(xy 264.16 177.8) (xy 274.32 177.8)
 		)
 		(stroke
@@
 	(wire
 		(pts
+			(xy 287.02 170.18) (xy 289.56 170.18)
+		)
+		(stroke
+			(width 0)
+			(type default)
+		)
+	)
+	(wire
+		(pts
 			(xy 144.78 236.22) (xy 147.32 236.22)
 		)
@@
 	(wire
 		(pts
-			(xy 264.16 170.18) (xy 269.24 170.18)
+			(xy 264.16 170.18) (xy 279.4 170.18)
 		)
 		(stroke
@@
 	)
 	(label "d8"
-		(at 269.24 177.8 0)
+		(at 284.48 177.8 0)
 		(fields_autoplaced yes)
 		(effects
@@
 		)
 	)
+	(label "tx"
+		(at 289.56 170.18 0)
+		(fields_autoplaced yes)
+		(effects
+			(font
+				(size 1.27 1.27)
+			)
+			(justify left bottom)
+		)
+	)
 	(label "conn2-2"
 		(at 265.43 193.04 0)
@@
 	)
 	(symbol
+		(lib_id "models:R-10k")
+		(at 283.21 170.18 90)
+		(unit 1)
+		(exclude_from_sim no)
+		(in_bom yes)
+		(on_board yes)
+		(dnp no)
+		(property "Reference" "R12-10k5"
+			(at 283.21 168.148 90)
+			(effects
+				(font
+					(size 1.27 1.27)
+				)
+			)
+		)
+		(property "Value" "R-1k"
+			(at 283.464 170.18 90)
+			(effects
+				(font
+					(size 1.27 1.27)
+				)
+			)
+		)
+		(property "Footprint" "Resistor_SMD:R_0805_2012Metric"
+			(at 283.21 171.958 90)
+			(effects
+				(font
+					(size 1.27 1.27)
+				)
+				(hide yes)
+			)
+		)
+		(property "Datasheet" "~"
+			(at 283.21 170.18 0)
+			(effects
+				(font
+					(size 1.27 1.27)
+				)
+				(hide yes)
+			)
+		)
+		(property "Description" "Resistor"
+			(at 283.21 170.18 0)
+			(effects
+				(font
+					(size 1.27 1.27)
+				)
+				(hide yes)
+			)
+		)
+		(property "LCSC Part" "C17414"
+			(at 283.21 170.18 0)
+			(effects
+				(font
+					(size 1.27 1.27)
+				)
+				(hide yes)
+			)
+		)
+		(property "Supplier" "LCSCRef"
+			(at 283.21 170.18 0)
+			(effects
+				(font
+					(size 1.27 1.27)
+				)
+				(hide yes)
+			)
+		)
+		(pin "1"
+		)
+		(pin "2"
+		)
+		(instances
+			(project "IoTmanager-v2"
+				(path "/e30adb8f-2050-4707-a23b-b56498f87e6f"
+					(reference "R12-10k5")
+					(unit 1)
+				)
+			)
+		)
+	)
+	(symbol
 		(lib_id "power:+5C")
 		(at 123.19 41.91 0)
@@
 			)
 		)
-		(property "Value" "R-1k"
+		(property "Value" "R-4k7"
 			(at 148.59 170.18 90)
 			(effects
@@
 			)
 		)
-		(property "Value" "R-1k"
+		(property "Value" "R-4k7"
 			(at 148.59 167.64 90)
 			(effects
@@
 					(unit 1)
 				)
+			)
+		)
+	)
+	(symbol
+		(lib_id "models:R-10k")
+		(at 278.13 177.8 90)
+		(unit 1)
+		(exclude_from_sim no)
+		(in_bom yes)
+		(on_board yes)
+		(dnp no)
+		(property "Reference" "R12-10k4"
+			(at 278.13 175.768 90)
+			(effects
+				(font
+					(size 1.27 1.27)
+				)
+			)
+		)
+		(property "Value" "R-1k"
+			(at 278.13 177.8 90)
+			(effects
+				(font
+					(size 1.27 1.27)
+				)
+			)
+		)
+		(property "Footprint" "Resistor_SMD:R_0805_2012Metric"
+			(at 278.13 179.578 90)
+			(effects
+				(font
+					(size 1.27 1.27)
+				)
+				(hide yes)
+			)
+		)
+		(property "Datasheet" "~"
+			(at 278.13 177.8 0)
+			(effects
+				(font
+					(size 1.27 1.27)
+				)
+				(hide yes)
+			)
+		)
+		(property "Description" "Resistor"
+			(at 278.13 177.8 0)
+			(effects
+				(font
+					(size 1.27 1.27)
+				)
+				(hide yes)
+			)
+		)
+		(property "LCSC Part" "C17414"
+			(at 278.13 177.8 0)
+			(effects
+				(font
+					(size 1.27 1.27)
+				)
+				(hide yes)
+			)
+		)
+		(property "Supplier" "LCSCRef"
+			(at 278.13 177.8 0)
+			(effects
+				(font
+					(size 1.27 1.27)
+				)
+				(hide yes)
+			)
+		)
+		(pin "1"
+		)
+		(pin "2"
+		)
+		(instances
+			(project "IoTmanager-v2"
+				(path "/e30adb8f-2050-4707-a23b-b56498f87e6f"
+					(reference "R12-10k4")
+					(unit 1)
+				)

Commit message: update
Parts:
- dc-in1: footprint module-custom-for-esp8266:dc-in-plastic-standard -> module-custom-for-esp8266:5.5PowerIn; symbol models:c-in-plastic-standard -> models:5.5powerIn; Availability (none) -> In Stock; Check_prices (none) -> https://www.snapeda.com/parts/54-00133/Tensility/view-part/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; Description_1 (none) -> Connector, dc jack 5.5x2.1 mm, PCB mount, 90 degrees, silve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; MANUFACTURER (none) -> TENSILITY; MAXIMUM_PACKAGE_HEIGHT (none) -> 10.8mm; MF (none) -> Tensility International Corp; MP (none) -> 54-00133; PARTREV (none) -> A; Package (none) -> None; Price (none) -> None; SNAPEDA_PN (none) -> 54-00133; STANDARD (none) -> Manufacturer Recommendations; SnapEDA_Link (none) -> https://www.snapeda.com/parts/54-00133/Tensility/view-part/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
Connections:
- net +12C: now also dc-in1.A; no longer dc-in1.1 (+12)
- net GNDPWR: now also dc-in1.B, dc-in1.C; no longer dc-in1.3 (GND)

Commit message: update
Parts:
- U8: value MMDT4413-7-F -> MMDT4413
Other:
- moved on the sheet: R21
Changed lines of the file:
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@@
 	(wire
 		(pts
-			(xy 20.32 245.11) (xy 38.1 245.11)
-		)
-		(stroke
-			(width 0)
-			(type default)
-		)
-	)
-	(wire
-		(pts
 			(xy 87.63 245.11) (xy 87.63 307.34)
 		)
@@
 	(wire
 		(pts
-			(xy 76.2 266.7) (xy 76.2 270.51)
+			(xy 38.1 288.29) (xy 38.1 292.1)
 		)
 		(stroke
@@
 	(wire
 		(pts
-			(xy 20.32 266.7) (xy 20.32 245.11)
-		)
-		(stroke
-			(width 0)
-			(type default)
-		)
-	)
-	(wire
-		(pts
 			(xy 115.57 232.41) (xy 125.73 232.41)
 		)
@@
 	(wire
 		(pts
-			(xy 24.13 264.16) (xy 25.4 264.16)
+			(xy 40.64 269.24) (xy 40.64 270.51)
 		)
 		(stroke
@@
 	(wire
 		(pts
-			(xy 25.4 259.08) (xy 25.4 261.62)
+			(xy 43.18 256.54) (xy 43.18 270.51)
 		)
 		(stroke
@@
 	(wire
 		(pts
-			(xy 11.43 264.16) (xy 16.51 264.16)
+			(xy 40.64 256.54) (xy 40.64 261.62)
 		)
 		(stroke
@@
 	(wire
 		(pts
-			(xy 25.4 266.7) (xy 20.32 266.7)
-		)
-		(stroke
-			(width 0)
-			(type default)
-		)
-	)
-	(wire
-		(pts
 			(xy 102.87 157.48) (xy 102.87 175.26)
 		)
@@
 	(wire
 		(pts
+			(xy 40.64 288.29) (xy 43.18 288.29)
+		)
+		(stroke
+			(width 0)
+			(type default)
+		)
+	)
+	(wire
+		(pts
 			(xy 165.1 109.22) (xy 168.91 109.22)
 		)
@@
 	(wire
 		(pts
-			(xy 76.2 261.62) (xy 76.2 264.16)
-		)
-		(stroke
-			(width 0)
-			(type default)
-		)
-	)
-	(wire
-		(pts
 			(xy 102.87 186.69) (xy 90.17 186.69)
 		)
@@
 	(wire
 		(pts
+			(xy 38.1 245.11) (xy 38.1 270.51)
+		)
+		(stroke
+			(width 0)
+			(type default)
+		)
+	)
+	(wire
+		(pts
 			(xy 193.04 237.49) (xy 193.04 241.3)
 		)
@@
 	)
 	(label "d3"
-		(at 11.43 264.16 0)
+		(at 40.64 256.54 270)
 		(fields_autoplaced yes)
 		(effects
@@
 				(size 1.27 1.27)
 			)
-			(justify left bottom)
+			(justify right bottom)
 		)
 	)
@@
 	(symbol
 		(lib_id "models:R-1k")
-		(at 20.32 264.16 270)
+		(at 40.64 265.43 180)
 		(unit 1)
 		(exclude_from_sim no)
@@
 		(dnp no)
 		(property "Reference" "R21"
-			(at 20.32 259.842 90)
+			(at 44.958 265.43 90)
 			(effects
 				(font
@@
 		)
 		(property "Value" "R-1k"
-			(at 20.574 261.62 90)
+			(at 43.18 265.684 90)
 			(effects
 				(font
@@
 		)
 		(property "Footprint" "Resistor_SMD:R_0805_2012Metric"
-			(at 20.32 262.382 90)
+			(at 42.418 265.43 90)
 			(effects
 				(font
@@
 		)
 		(property "Datasheet" "~"
-			(at 20.32 264.16 0)
+			(at 40.64 265.43 0)
 			(effects
 				(font
@@
 		)
 		(property "Description" "Resistor"
-			(at 20.32 264.16 0)
+			(at 40.64 265.43 0)
 			(effects
 				(font
@@
 		)
 		(property "LCSC Part" "C25905"
-			(at 20.32 264.16 0)
+			(at 40.64 265.43 0)
 			(effects
 				(font
@@
 		)
 		(property "Supplier" "LCSCRef"
-			(at 20.32 264.16 0)
+			(at 40.64 265.43 0)
 			(effects
 				(font
@@
 					(size 1.27 1.27)
 				)
+				(hide yes)
 			)
 		)
@@
 					(size 1.27 1.27)
 				)
+				(hide yes)
 			)
 		)
@@
 	(symbol
 		(lib_id "power:+3.3V")
-		(at 25.4 259.08 0)
+		(at 43.18 256.54 0)
 		(unit 1)
 		(exclude_from_sim no)
@@
 		(fields_autoplaced yes)
 		(property "Reference" "#PWR062"
-			(at 25.4 262.89 0)
+			(at 43.18 260.35 0)
 			(effects
 				(font
@@
 		)
 		(property "Value" "+3.3V"
-			(at 25.4 254 0)
+			(at 43.18 251.46 0)
 			(effects
 				(font
@@
 		)
 		(property "Footprint" ""
-			(at 25.4 259.08 0)
+			(at 43.18 256.54 0)
 			(effects
 				(font
@@
 		)
 		(property "Datasheet" ""
-			(at 25.4 259.08 0)
+			(at 43.18 256.54 0)
 			(effects
 				(font
@@
 		)
 		(property "Description" "Power symbol creates a global label with name \"+3.3V\""
-			(at 25.4 259.08 0)
+			(at 43.18 256.54 0)
 			(effects
 				(font
@@
 		)
 		(property "Footprint" "module-custom-for-esp8266:PJ-320A"
-			(at 35.56 151.13 0)
+			(at 40.132 158.242 0)
 			(effects
 				(font
@@
 		(dnp no)
 		(property "Reference" "R12-10k3"
-			(at 148.59 168.148 90)
+			(at 156.972 173.482 90)
 			(effects
 				(font
 					(size 1.27 1.27)
 				)
+				(hide yes)
 			)
 		)
 		(property "Value" "R-4k7"
-			(at 148.59 170.18 90)
+			(at 149.098 173.228 90)
 			(effects
 				(font
@@
 	)
 	(symbol
+		(lib_name "MMDT4413-7-F_1")
 		(lib_id "models:MMDT4413-7-F")
-		(at 76.2 266.7 180)
+		(at 25.4 281.94 0)
 		(unit 1)
 		(exclude_from_sim no)
@@
 		(fields_autoplaced yes)
 		(property "Reference" "U8"
-			(at 50.8 251.46 0)
+			(at 48.26 278.1299 0)
 			(effects
 				(font
 					(size 1.524 1.524)
 				)
+				(justify left)
 			)
 		)
-		(property "Value" "MMDT4413-7-F"
-			(at 50.8 254 0)
+		(property "Value" "MMDT4413"
+			(at 48.26 280.6699 0)
 			(effects
 				(font
 					(size 1.524 1.524)
 				)
+				(justify left)
 			)
 		)
 		(property "Footprint" "module-custom-for-esp8266:SOT-363_DIO"
-			(at 76.2 266.7 0)
+			(at 40.64 295.91 0)
 			(effects
 				(font
@@
 		)
 		(property "Datasheet" "MMDT4413-7-F"
-			(at 76.2 266.7 0)
+			(at 41.91 293.37 0)
 			(effects
 				(font
@@
 		)
 		(property "Description" ""
-			(at 76.2 266.7 0)
+			(at 38.1 288.29 90)
 			(effects
 				(font
@@
 		(dnp no)
 		(property "Reference" "R12-10k2"
-			(at 148.59 165.608 90)
+			(at 153.416 164.592 90)
 			(effects
 				(font
 					(size 1.27 1.27)
 				)
+				(hide yes)
 			)
 		)
 		(property "Value" "R-4k7"
-			(at 148.59 167.64 90)
+			(at 150.622 165.1 90)
 			(effects
 				(font
@@
 					(size 1.27 1.27)
 				)
+				(hide yes)
 			)
 		)
@@
 	(symbol
 		(lib_id "power:GNDPWR")
-		(at 76.2 270.51 0)
+		(at 38.1 292.1 0)
 		(unit 1)
 		(exclude_from_sim no)
@@
 		(fields_autoplaced yes)
 		(property "Reference" "#PWR061"
-			(at 76.2 275.59 0)
+			(at 38.1 297.18 0)
 			(effects
 				(font
@@
 		)
 		(property "Value" "GNDPWR"
-			(at 76.073 274.32 0)
+			(at 37.973 295.91 0)
 			(effects
 				(font
@@
 		)
 		(property "Footprint" ""
-			(at 76.2 271.78 0)
+			(at 38.1 293.37 0)
 			(effects
 				(font
@@
 		)
 		(property "Datasheet" ""
-			(at 76.2 271.78 0)
+			(at 38.1 293.37 0)
 			(effects
 				(font
@@
 		)
 		(property "Description" "Power symbol creates a global label with name \"GNDPWR\" , global ground"
-			(at 76.2 270.51 0)
+			(at 38.1 292.1 0)
 			(effects
 				(font

Commit message: update
Parts:
- removed R3: R-100, Resistor_SMD:R_0805_2012Metric, symbol models:R-100
- added C4: C_Polarized_10uF, Capacitor_THT:CP_Radial_D10.0mm_P3.50mm, symbol resistor:C_Polarized_Small
Connections:
- net +3.3V: now also RV1.1
- net GNDPWR: now also C4.2; no longer U5.1 (Sleeve)
- net a0: now also U5.1 (Sleeve)
- net at RV1.2: now also U5.2 (Tip), C4.1
- removed net a0-in-res: RV1.1, U5.2 (Tip)
Other:
- moved on the sheet: RV1, U5

Commit message: auto update from EPAM computer
Parts:
- removed RV1: res-a0, Potentiometer_THT:Potentiometer_Bourns_3296W_Vertical, symbol Device:R_Potentiometer
- added 33R1: 33R, Resistor_SMD:R_0805_2012Metric, symbol models:R-10k
- added R10-10k2, R10-10k3: R-10k, Resistor_SMD:R_0805_2012Metric, symbol models:R-10k
Connections:
- net +3.3V: now also R10-10k2.1
- net GNDPWR: now also R10-10k3.2
- net a0: now also 33R1.2
- net at C4.1, U5.2 (Tip): now also 33R1.1, R10-10k2.2, R10-10k3.1

Commit message: update
Parts:
- added J1: powerRelay, Connector_PinHeader_2.54mm:PinHeader_1x02_P2.54mm_Vertical, symbol Connector:Conn_01x02_Pin
Connections:
- net +5C: now also J1.1 (Pin_1); no longer D2.1 (K), D3.1 (K), D4.1 (K), D5.1 (K), K3.A1, K5.A1, K6.A1, K7.A1
- new net pwrRel: D2.1 (K), D3.1 (K), D4.1 (K), D5.1 (K), J1.2 (Pin_2), K3.A1, K5.A1, K6.A1, K7.A1

Commit message: update
Parts:
- removed R21: R-1k, Resistor_SMD:R_0805_2012Metric, symbol models:R-1k
- removed U10, U11, U9: MMDT4413-7-F, module-custom-for-esp8266:SOT-363_DIO, symbol models:MMDT4413-7-F
- removed U8: MMDT4413, module-custom-for-esp8266:SOT-363_DIO, symbol models:MMDT4413-7-F
- added Q1, Q3, Q5, Q7: MMBT5401, Package_TO_SOT_SMD:SOT-23, symbol models:MMBT5401-pnp
- added Q2, Q4, Q6, Q8: MMBT5551-npn, Package_TO_SOT_SMD:SOT-23, symbol models:MMBT5551-npn
- added R15, R17, R18, R19, R3: R-1k, Resistor_SMD:R_0805_2012Metric, symbol models:R-1k
Connections:
- net +12C: now also J2.2 (Pin_2); no longer J2.3 (Pin_3)
- net +3.3V: now also J2.4 (Pin_4), Q1.2 (E), Q3.2 (E), Q5.2 (E), Q7.2 (E); no longer J2.5 (Pin_5)
- net +5C: now also J2.3 (Pin_3); no longer J2.4 (Pin_4)
- net GNDPWR: now also Q2.2 (E), Q4.2 (E), Q6.2 (E), Q8.2 (E); no longer J2.2 (Pin_2)
- net d0: now also R15.2; no longer R4.2
- net d3: now also R3.2
- net d4: now also J2.8 (Pin_8), R18.2
- net mosf1-out-d5: now also J2.5 (Pin_5); no longer J2.6 (Pin_6)
- net mosf2-out-d6: now also J2.6 (Pin_6); no longer J2.7 (Pin_7)
- net mosf3-out-d7: now also J2.7 (Pin_7); no longer J2.8 (Pin_8)
- net rx: no longer R14.2
- net at R12.1: now also Q3.1 (B)
- net at R4.1: now also Q2.1 (B)
- net at D5.2 (A), K7.A2: now also Q8.3 (C)
- net at D3.2 (A), K5.A2: now also Q4.3 (C)
- net at R14.1: now also Q4.1 (B)
- net at D4.2 (A), K6.A2: now also Q6.3 (C)
- net at D2.2 (A), K3.A2: now also Q2.3 (C)
- new net: Q3.3 (C), R14.2
- new net: Q7.1 (B), R18.1
- new net: Q8.1 (B), R19.1
- new net: Q1.1 (B), R3.1
- new net: Q7.3 (C), R19.2
- new net: Q6.1 (B), R17.1
- new net: Q5.1 (B), R15.1
- new net: Q5.3 (C), R17.2
- new net: Q1.3 (C), R4.2
