File: IoTmanager/IoTmanager-v2.kicad_pcb (KiCad board)
At the start: 2 copper layers, 50 x 70.7 mm, 57 parts, among them J1 prog, J2 Conn_01x12_Pin, J3 Conn_01x12_Pin, J4 flash, J5 reset, K3 ZC32F-012-HS3-copy, K5 ZC32F-012-HS3-copy, K6 ZC32F-012-HS3-copy, K7 ZC32F-012-HS3-copy, Q1 MMBT5401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

Commit message: update
Parts:
- removed J1: prog, Connector_PinHeader_2.54mm:PinHeader_1x04_P2.54mm_Vertical
- removed J4: flash, Connector_PinHeader_2.54mm:PinHeader_1x02_P2.54mm_Vertical
- removed Q1, Q10, Q8: MMBT5401, Package_TO_SOT_SMD:SOT-23
- removed Q11, Q7: MMBT5551-npn, Package_TO_SOT_SMD:SOT-23
- removed R10, R11, R12: R-10k, Resistor_SMD:R_0805_2012Metric
- removed U3: TSOP23xx, OptoDevice:Vishay_MOLD-3Pin
- added J4-flash1: flash, Connector_PinHeader_2.54mm:PinHeader_1x02_P2.54mm_Vertical, F.Cu at (113.6, 100.7)
- added Q1-pnp1: MMBT5401, Package_TO_SOT_SMD:SOT-23, B.Cu at (93.1, 88.5)
- added Q10-pnp1: MMBT5401, Package_TO_SOT_SMD:SOT-23, B.Cu at (113.5, 88.7)
- added Q11-npn1: MMBT5551-npn, Package_TO_SOT_SMD:SOT-23, B.Cu at (113.6, 94.4)
- added Q7-npn1: MMBT5551-npn, Package_TO_SOT_SMD:SOT-23, B.Cu at (93.0, 94.4)
- added Q8-pnp1: MMBT5401, Package_TO_SOT_SMD:SOT-23, B.Cu at (103.4, 89.0)
- added R10-10k1: R-10k, Resistor_SMD:R_0805_2012Metric, B.Cu at (97.6, 111.0)
- added R11-10k1: R-10k, Resistor_SMD:R_0805_2012Metric, B.Cu at (101.1, 110.7)
- added R12-10k1: R-10k, Resistor_SMD:R_0805_2012Metric, B.Cu at (86.8, 88.0)
- added U3-tsop23: TSOP23xx, OptoDevice:Vishay_MOLD-3Pin, F.Cu at (81.7, 118.9)
- added prog1: prog, Connector_PinHeader_2.54mm:PinHeader_1x04_P2.54mm_Vertical, F.Cu at (88.6, 108.3)
- K3, K5, K6, K7: footprint module-custom-for-esp8266:ZC32F-012-HS3 -> module-custom-for-esp8266:HF32F-005-ZS3
- moved K6 14.5 mm to (98.7, 98.8)
- moved K3 14.5 mm to (78.0, 98.8)
- moved K5 14.5 mm to (88.4, 98.8)
- moved K7 14.5 mm to (109.0, 98.7)
- moved R4 0.76 mm to (93.2, 85.3)

Commit message: update
Parts:
- added D2: 1N4148, module-custom-for-esp8266:sod80-1n1448, B.Cu at (81.9, 97.6)
- added D3: 1N4148, module-custom-for-esp8266:sod80-1n1448, B.Cu at (92.5, 97.7)
- added D4: 1N4148, module-custom-for-esp8266:sod80-1n1448, B.Cu at (102.6, 97.6)
- added D5: 1N4148, module-custom-for-esp8266:sod80-1n1448, B.Cu at (113.0, 97.7)

Commit message: update
Parts:
- added R7: R-4k7, Resistor_SMD:R_0805_2012Metric, B.Cu at (118.1, 124.0)
- moved U12 0.78 mm to (113.0, 76.9)
- moved C1 0.76 mm to (86.9, 74.4)
- moved U4 0.56 mm to (105.4, 68.0)
Changed lines of the file:
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@@
 	(footprint "module-custom-for-esp8266:Mini360_step-down"
 		(layer "F.Cu")
-		(at 105.52 68.52 180)
+		(at 105.41 67.9704 180)
 		(property "Reference" "U4"
 			(at 0 0.5 0)
@@
 	(footprint "Capacitor_THT:CP_Radial_D10.0mm_P3.50mm"
 		(layer "F.Cu")
-		(at 86.926723 75.184)
+		(at 86.8732 74.422)
 		(descr "CP, Radial series, Radial, pin pitch=3.50mm, , diameter=10mm, Electrolytic Capacitor")
 		(tags "CP Radial series Radial pin pitch 3.50mm  diameter 10mm Electrolytic Capacitor")
@@
 		)
 	)
+	(footprint "Resistor_SMD:R_0805_2012Metric"
+		(layer "B.Cu")
+		(at 118.0592 123.952)
+		(descr "Resistor SMD 0805 (2012 Metric), square (rectangular) end terminal, IPC_7351 nominal, (Body size source: IPC-SM-782 page 72, https://www.pcb-3d.com/wordpress/wp-content/uploads/ipc-sm-782a_amendment_1_and_2.pdf), generated with kicad-footprint-generator")
+		(tags "resistor")
+		(property "Reference" "R7"
+			(at 2.6924 0.1016 0)
+			(layer "B.SilkS")
+			(effects
+				(font
+					(size 1 1)
+					(thickness 0.15)
+				)
+				(justify mirror)
+			)
+		)
+		(property "Value" "R-4k7"
+			(at 0 -1.65 0)
+			(layer "B.Fab")
+			(effects
+				(font
+					(size 1 1)
+					(thickness 0.15)
+				)
+				(justify mirror)
+			)
+		)
+		(property "Footprint" "Resistor_SMD:R_0805_2012Metric"
+			(at 0 0 180)
+			(unlocked yes)
+			(layer "B.Fab")
+			(hide yes)
+			(effects
+				(font
+					(size 1.27 1.27)
+					(thickness 0.15)
+				)
+				(justify mirror)
+			)
+		)
+		(property "Datasheet" ""
+			(at 0 0 180)
+			(unlocked yes)
+			(layer "B.Fab")
+			(hide yes)
+			(effects
+				(font
+					(size 1.27 1.27)
+					(thickness 0.15)
+				)
+				(justify mirror)
+			)
+		)
+		(property "Description" "Resistor"
+			(at 0 0 180)
+			(unlocked yes)
+			(layer "B.Fab")
+			(hide yes)
+			(effects
+				(font
+					(size 1.27 1.27)
+					(thickness 0.15)
+				)
+				(justify mirror)
+			)
+		)
+		(property "JLCPCB Part" "C25905"
+			(at 0 0 180)
+			(unlocked yes)
+			(layer "B.Fab")
+			(hide yes)
+			(effects
+				(font
+					(size 1 1)
+					(thickness 0.15)
+				)
+				(justify mirror)
+			)
+		)
+		(property ki_fp_filters "R_*")
+		(sheetname "Корневой лист")
+		(sheetfile "IoTmanager-v2.kicad_sch")
+		(attr smd)
+		(fp_line
+			(start 0.227064 -0.735)
+			(end -0.227064 -0.735)
+			(stroke
+				(width 0.12)
+				(type solid)
+			)
+			(layer "B.SilkS")
+		)
+		(fp_line
+			(start 0.227064 0.735)
+			(end -0.227064 0.735)
+			(stroke
+				(width 0.12)
+				(type solid)
+			)
+			(layer "B.SilkS")
+		)
+		(fp_line
+			(start -1.68 -0.95)
+			(end 1.68 -0.95)
+			(stroke
+				(width 0.05)
+				(type solid)
+			)
+			(layer "B.CrtYd")
+		)
+		(fp_line
+			(start -1.68 0.95)
+			(end -1.68 -0.95)
+			(stroke
+				(width 0.05)
+				(type solid)
+			)
+			(layer "B.CrtYd")
+		)
+		(fp_line
+			(start 1.68 -0.95)
+			(end 1.68 0.95)
+			(stroke
+				(width 0.05)
+				(type solid)
+			)
+			(layer "B.CrtYd")
+		)
+		(fp_line
+			(start 1.68 0.95)
+			(end -1.68 0.95)
+			(stroke
+				(width 0.05)
+				(type solid)
+			)
+			(layer "B.CrtYd")
+		)
+		(fp_line
+			(start -1 -0.625)
+			(end 1 -0.625)
+			(stroke
+				(width 0.1)
+				(type solid)
+			)
+			(layer "B.Fab")
+		)
+		(fp_line
+			(start -1 0.625)
+			(end -1 -0.625)
+			(stroke
+				(width 0.1)
+				(type solid)
+			)
+			(layer "B.Fab")
+		)
+		(fp_line
+			(start 1 -0.625)
+			(end 1 0.625)
+			(stroke
+				(width 0.1)
+				(type solid)
+			)
+			(layer "B.Fab")
+		)
+		(fp_line
+			(start 1 0.625)
+			(end -1 0.625)
+			(stroke
+				(width 0.1)
+				(type solid)
+			)
+			(layer "B.Fab")
+		)
+		(fp_text user "${REFERENCE}"
+			(at 0 0 0)
+			(layer "B.Fab")
+			(effects
+				(font
+					(size 0.5 0.5)
+					(thickness 0.08)
+				)
+				(justify mirror)
+			)
+		)
+		(pad "1" smd roundrect
+			(at -0.9125 0)
+			(size 1.025 1.4)
+			(layers "B.Cu" "B.Paste" "B.Mask")
+			(roundrect_rratio 0.243902)
+			(net 32 "/d7")
+			(pintype "passive")
+		)
+		(pad "2" smd roundrect
+			(at 0.9125 0)
+			(size 1.025 1.4)
+			(layers "B.Cu" "B.Paste" "B.Mask")
+			(roundrect_rratio 0.243902)
+			(net 17 "+5C")
+			(pintype "passive")
+		)
+		(model "${KICAD8_3DMODEL_DIR}/Resistor_SMD.3dshapes/R_0805_2012Metric.wrl"
+			(offset
+				(xyz 0 0 0)
+			)
+			(scale
+				(xyz 1 1 1)
+			)
+			(rotate
+				(xyz 0 0 0)
+			)
+		)
+	)
 	(footprint "Package_TO_SOT_SMD:TO-252-2"
 		(layer "B.Cu")
@@
 	(footprint "Package_TO_SOT_SMD:SOT-223-3_TabPin2"
 		(layer "B.Cu")
-		(at 113.19 76.11)
+		(at 112.9792 76.8604)
 		(descr "module CMS SOT223 4 pins")
 		(tags "CMS SOT")
 		(property "Reference" "U12"
-			(at 0.0432 4.4588 0)
+			(at 0.0432 4.4588 360)
 			(layer "B.SilkS")
 			(effects
@@
 		)
 		(property "Value" "AMS1117-5.0"
-			(at 0.31 -4.22 0)
+			(at 0.31 -4.22 360)
 			(layer "B.Fab")
 			(effects

Commit message: update
Connections:
- R7 pad 1: /d7 -> /d2
- U7 pad 2: /d7 -> /d2
Changed lines of the file:
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@@
 			(layers "*.Cu" "*.Mask")
 			(remove_unused_layers no)
-			(net 32 "/d7")
+			(net 16 "/d2")
 			(pinfunction "DQ")
 			(pintype "bidirectional")
@@
 			(layers "B.Cu" "B.Paste" "B.Mask")
 			(roundrect_rratio 0.243902)
-			(net 32 "/d7")
+			(net 16 "/d2")
 			(pintype "passive")
 		)
@@
 		(tags "CMS SOT")
 		(property "Reference" "U12"
-			(at 0.0432 4.4588 360)
+			(at 0.0432 4.4588 0)
 			(layer "B.SilkS")
 			(effects
@@
 		)
 		(property "Value" "AMS1117-5.0"
-			(at 0.31 -4.22 360)
+			(at 0.31 -4.22 0)
 			(layer "B.Fab")
 			(effects

Commit message: update
Connections:
- C1 pad 1: +5C -> +3.3V
Changed lines of the file:
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@@
 			(layers "*.Cu" "*.Mask")
 			(remove_unused_layers no)
-			(net 17 "+5C")
+			(net 22 "+3.3V")
 			(pintype "passive")
 		)

Commit message: update
Parts:
- U7: footprint Package_TO_SOT_THT:TO-92_Inline -> Connector_PinHeader_2.54mm:PinHeader_1x03_P2.54mm_Vertical
- moved R12-10k1 20.7 mm to (85.5, 108.7)
- moved prog1 7.57 mm to (89.0, 115.9), turned to 180 degrees
- moved R7 3.36 mm to (121.4, 123.8)
- moved Q10-pnp1 1.38 mm to (114.3, 87.6)
- moved Q11-npn1 1.38 mm to (114.4, 93.3)
- moved R25 1.38 mm to (114.2, 84.9)
- moved R26 1.38 mm to (114.2, 90.3)
- moved Q5 1.30 mm to (83.3, 87.6)
- moved Q6 1.30 mm to (83.3, 93.0)
- moved R21 1.30 mm to (83.1, 84.9)
- moved R22 1.30 mm to (83.1, 90.3)
- moved R17 0.93 mm to (93.2, 90.6)
- moved Q1-pnp1 0.93 mm to (93.5, 87.7)
- moved Q7-npn1 0.93 mm to (93.4, 93.5)
- moved Q8-pnp1 0.92 mm to (104.0, 88.3)
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
Commit message: update
Parts:
- moved J5 2.75 mm to (111.0, 103.7), turned to 90 degrees
Changed lines of the file:
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@@
 		)
 		(fp_text user "${REFERENCE}"
-			(at 0 2.54 360)
+			(at 0 2.54 0)
 			(layer "F.Fab")
 			(effects
@@
 	(footprint "Connector_PinHeader_2.54mm:PinHeader_1x02_P2.54mm_Vertical"
 		(layer "F.Cu")
-		(at 113.665 104.53 -90)
+		(at 111.0438 103.6828 90)
 		(descr "Through hole straight pin header, 1x02, 2.54mm pitch, single row")
 		(tags "Through hole pin header THT 1x02 2.54mm single row")
@@
 		)
 		(property "Footprint" "Connector_PinHeader_2.54mm:PinHeader_1x02_P2.54mm_Vertical"
-			(at 0 0 -90)
+			(at 0 0 90)
 			(unlocked yes)
 			(layer "F.Fab")
@@
 		)
 		(property "Datasheet" ""
-			(at 0 0 -90)
+			(at 0 0 90)
 			(unlocked yes)
 			(layer "F.Fab")
@@
 		)
 		(property "Description" "Generic connector, single row, 01x02, script generated"
-			(at 0 0 -90)
+			(at 0 0 90)
 			(unlocked yes)
 			(layer "F.Fab")
@@
 		)
 		(property "Supplier" ""
-			(at 0 0 -90)
+			(at 0 0 90)
 			(unlocked yes)
 			(layer "F.Fab")
@@
 		(attr through_hole)
 		(fp_line
-			(start -1.33 3.87)
-			(end 1.33 3.87)
+			(start -1.33 -1.33)
+			(end 0 -1.33)
 			(stroke
 				(width 0.12)
@@
 		)
 		(fp_line
-			(start -1.33 1.27)
-			(end -1.33 3.87)
+			(start -1.33 0)
+			(end -1.33 -1.33)
 			(stroke
 				(width 0.12)
@@
 		)
 		(fp_line
-			(start -1.33 1.27)
-			(end 1.33 1.27)
+			(start 1.33 1.27)
+			(end 1.33 3.87)
 			(stroke
 				(width 0.12)
@@
 		)
 		(fp_line
-			(start 1.33 1.27)
-			(end 1.33 3.87)
+			(start -1.33 1.27)
+			(end 1.33 1.27)
 			(stroke
 				(width 0.12)
@@
 		)
 		(fp_line
-			(start -1.33 0)
-			(end -1.33 -1.33)
+			(start -1.33 1.27)
+			(end -1.33 3.87)
 			(stroke
 				(width 0.12)
@@
 		)
 		(fp_line
-			(start -1.33 -1.33)
-			(end 0 -1.33)
+			(start -1.33 3.87)
+			(end 1.33 3.87)
 			(stroke
 				(width 0.12)
@@
 		)
 		(fp_line
-			(start -1.8 4.35)
-			(end 1.8 4.35)
+			(start 1.8 -1.8)
+			(end -1.8 -1.8)
 			(stroke
 				(width 0.05)
@@
 		)
 		(fp_line
-			(start 1.8 4.35)
-			(end 1.8 -1.8)
+			(start -1.8 -1.8)
+			(end -1.8 4.35)
 			(stroke
 				(width 0.05)
@@
 		)
 		(fp_line
-			(start -1.8 -1.8)
-			(end -1.8 4.35)
+			(start 1.8 4.35)
+			(end 1.8 -1.8)
 			(stroke
 				(width 0.05)
@@
 		)
 		(fp_line
-			(start 1.8 -1.8)
-			(end -1.8 -1.8)
+			(start -1.8 4.35)
+			(end 1.8 4.35)
 			(stroke
 				(width 0.05)
@@
 		)
 		(fp_line
-			(start -1.27 3.81)
-			(end -1.27 -0.635)
+			(start 1.27 -1.27)
+			(end 1.27 3.81)
 			(stroke
 				(width 0.1)
@@
 		)
 		(fp_line
-			(start 1.27 3.81)
-			(end -1.27 3.81)
+			(start -0.635 -1.27)
+			(end 1.27 -1.27)
 			(stroke
 				(width 0.1)
@@
 		)
 		(fp_line
-			(start -0.635 -1.27)
-			(end 1.27 -1.27)
+			(start 1.27 3.81)
+			(end -1.27 3.81)
 			(stroke
 				(width 0.1)
@@
 		)
 		(fp_line
-			(start 1.27 -1.27)
-			(end 1.27 3.81)
+			(start -1.27 3.81)
+			(end -1.27 -0.635)
 			(stroke
 				(width 0.1)
@@
 		)
 		(fp_text user "${REFERENCE}"
-			(at 0 1.27 0)
+			(at 0 1.27 360)
 			(layer "F.Fab")
 			(effects
@@
 		)
 		(pad "1" thru_hole rect
-			(at 0 0 270)
+			(at 0 0 90)
 			(size 1.7 1.7)
 			(drill 1)
@@
 		)
 		(pad "2" thru_hole oval
-			(at 0 2.54 270)
+			(at 0 2.54 90)
 			(size 1.7 1.7)
 			(drill 1)

Commit message: update
Parts:
- added C2: C_Polarized_1000mF, Capacitor_THT:CP_Radial_D10.0mm_P3.50mm, F.Cu at (107.7, 73.2)
- added D6: LED, LED_THT:LED_D5.0mm, F.Cu at (82.7, 109.7)
- added R10: R-150, Resistor_SMD:R_0805_2012Metric, B.Cu at (84.0, 116.1)
- moved R16 16.5 mm to (103.1, 121.5)
- moved R12-10k1 12.2 mm to (97.3, 112.0)
- moved R3 7.86 mm to (105.2, 121.6)
- moved Jumper-d5 6.68 mm to (97.6, 77.9), turned to 90 degrees
- moved R9 4.04 mm to (83.2, 75.1)
- moved R2 3.27 mm to (100.9, 75.7)
- moved R13 2.90 mm to (97.2, 108.1)
- moved R1 2.88 mm to (102.5, 79.2), turned to 0 degrees
- moved R7 2.66 mm to (123.8, 122.6), turned to 90 degrees
- moved R10-10k1 2.36 mm to (99.7, 112.1)
- moved R11-10k1 1.65 mm to (102.0, 112.1)
- moved U12 1.30 mm to (114.2, 76.6)
- moved Jumper-d7 1.07 mm to (79.8, 77.4)
- moved Jumper-d6 0.87 mm to (90.1, 77.8)
- moved R23 0.74 mm to (104.1, 84.7)
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Connections:
- J2 pad 10: /conn1-9 -> /d1
- J2 pad 11: /conn1-10 -> /d2
- J2 pad 12: /d1 -> /d8
- J2 pad 2: +5C -> GNDPWR
- J2 pad 3: /rx -> +12C
- J2 pad 4: /tx -> +5C
- J2 pad 5: /d8 -> +3.3V
- J2 pad 9: /conn1-8 -> /d0
- J3 pad 10: /d2 -> /conn1-8
- J3 pad 11: /d0 -> /conn1-9
- J3 pad 12: GNDPWR -> /conn1-10
- R25 pad 2: /d4 -> /rx
- R7 pad 1: /d2 -> /d4
- U7 pad 2: /d2 -> /d4
