File: IoTmanager/IoTmanager-v2.kicad_pcb (KiCad board)
At the start: 2 copper layers, 48 x 75 mm, 62 parts, among them J2 Conn_01x12_Pin, J3 Conn_01x12_Pin, J4-flash1 flash, J5 reset, K3 ZC32F-012-HS3-copy, K5 ZC32F-012-HS3-copy, K6 ZC32F-012-HS3-copy, K7 ZC32F-012-HS3-copy, SW1 SW_PUSH_6mm_H4.3mm, U10 MMDT4413-7-F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

Commit message: update
Parts:
- dc-in1: footprint module-custom-for-esp8266:dc-in-plastic-standard -> module-custom-for-esp8266:5.5PowerIn
- moved R12-10k4 36.5 mm to (119.0, 121.8)
- moved C3 24.3 mm to (119.2, 75.6), turned to -90 degrees
- moved R16 13.2 mm to (118.8, 86.6)
- moved R1 11.0 mm to (104.9, 94.4)
- moved dc-in1 6.07 mm to (121.0, 68.3), turned to 90 degrees
- moved R12-10k2 5.92 mm to (107.8, 105.7)
- moved R13 4.41 mm to (113.9, 101.2)
- moved R7 3.02 mm to (120.3, 107.4)
- moved R6 2.59 mm to (107.8, 114.4), turned to 90 degrees
- moved D1 2.08 mm to (123.4, 82.7)
- moved RV1 2.08 mm to (122.8, 89.9)
- moved U3-tsop23 2.08 mm to (122.5, 79.4)
- moved C1 1.91 mm to (98.6, 119.1)
- moved C2 1.79 mm to (81.1, 119.1)
- moved Jumper-d6 1.35 mm to (107.2, 109.2)
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Routing:
- net /a0: vias 0 -> 1
- net (no net): vias 0 -> 2

Commit message: update
Parts:
- U8: value MMDT4413-7-F -> MMDT4413
Changed lines of the file:
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@@
 			)
 			(scale
-				(xyz 1 1 1)
+				(xyz 1 1 1.7)
 			)
 			(rotate
@@
 			)
 			(scale
-				(xyz 1 1 1)
+				(xyz 1 1 1.7)
 			)
 			(rotate
@@
 		(at 127.705 103.1 180)
 		(property "Reference" "U5"
-			(at 8.4455 -3.269 360)
+			(at 8.4455 -3.269 0)
 			(layer "F.SilkS")
 			(effects
@@
 		)
 		(property "Value" "PJ-320A"
-			(at 8.4455 -4.539 360)
+			(at 8.4455 -4.539 0)
 			(layer "F.Fab")
 			(effects
@@
 		)
 		(property "Footprint" "module-custom-for-esp8266:PJ-320A"
-			(at 0 0 360)
+			(at 0 0 0)
 			(layer "F.Fab")
 			(hide yes)
@@
 		)
 		(property "Datasheet" ""
-			(at 0 0 360)
+			(at 0 0 0)
 			(layer "F.Fab")
 			(hide yes)
@@
 		)
 		(property "Description" ""
-			(at 0 0 360)
+			(at 0 0 0)
 			(layer "F.Fab")
 			(hide yes)
@@
 		(tags "resistor")
 		(property "Reference" "Jumper-d5"
-			(at -1.85 0.26 360)
+			(at -1.85 0.26 0)
 			(layer "B.SilkS")
 			(hide yes)
@@
 		)
 		(property "Value" "1"
-			(at 2.5125 -0.6 360)
+			(at 2.5125 -0.6 0)
 			(layer "B.Fab")
 			(effects
@@
 		)
 		(fp_text user "${REFERENCE}"
-			(at 1.0125 0.3 360)
+			(at 1.0125 0.3 0)
 			(layer "B.Fab")
 			(effects
@@
 			)
 		)
-		(property "Value" "MMDT4413-7-F"
+		(property "Value" "MMDT4413"
 			(at -0.3 2.2 0)
 			(unlocked yes)

Commit message: update
Parts:
- removed R3: R-100, Resistor_SMD:R_0805_2012Metric
- added C4: C_Polarized_10uF, Capacitor_THT:CP_Radial_D10.0mm_P3.50mm, F.Cu at (108.1, 120.6)
- moved R6 38.7 mm to (78.5, 89.1), turned to -90 degrees
- moved R5 25.9 mm to (85.8, 94.7)
- moved Jumper-d6 22.6 mm to (89.9, 94.7)
- moved R8 9.71 mm to (105.8, 111.4), turned to -90 degrees
- moved G*** 6.21 mm to (111.9, 112.6)
- moved R12-10k2 1.34 mm to (107.2, 106.9), turned to 180 degrees
- moved R7 0.91 mm to (120.4, 108.3)
Connections:
- RV1 pad 1: /a0-in-res -> +3.3V
- RV1 pad 2: Net-(R3-Pad1) -> Net-(U5-Tip)
- U5 pad 1: GNDPWR -> /a0
- U5 pad 2: /a0-in-res -> Net-(U5-Tip)

Commit message: auto update from EPAM computer
Parts:
- removed RV1: res-a0, Potentiometer_THT:Potentiometer_Bourns_3296W_Vertical
- added 33R1: 33R, Resistor_SMD:R_0805_2012Metric, B.Cu at (120.9, 99.8)
- added R10-10k2: R-10k, Resistor_SMD:R_0805_2012Metric, B.Cu at (110.5, 101.4)
- added R10-10k3: R-10k, Resistor_SMD:R_0805_2012Metric, B.Cu at (106.0, 103.8)
- moved R12-10k2 4.67 mm to (110.6, 103.7)
- moved R10-10k1 1.28 mm to (106.2, 101.3)
- moved R8 0.74 mm to (105.5, 110.7)
- moved C3 0.53 mm to (119.5, 75.2)
- moved R13 0.35 mm to (114.2, 101.2)
- moved R7 0.32 mm to (120.3, 108.0)

Commit message: update
Parts:
- added J1: powerRelay, Connector_PinHeader_2.54mm:PinHeader_1x02_P2.54mm_Vertical, F.Cu at (121.3, 92.1)
- moved G*** 1.08 mm to (111.3, 111.7)
Connections:
- D2 pad 1: +5C -> /pwrRel
- D3 pad 1: +5C -> /pwrRel
- D4 pad 1: +5C -> /pwrRel
- D5 pad 1: +5C -> /pwrRel
- K3 pad A1: +5C -> /pwrRel
- K5 pad A1: +5C -> /pwrRel
- K6 pad A1: +5C -> /pwrRel
- K7 pad A1: +5C -> /pwrRel

Commit message: update
Parts:
- removed R21: R-1k, Resistor_SMD:R_0805_2012Metric
- removed U10, U11, U9: MMDT4413-7-F, module-custom-for-esp8266:SOT-363_DIO
- removed U8: MMDT4413, module-custom-for-esp8266:SOT-363_DIO
- added Q1: MMBT5401, Package_TO_SOT_SMD:SOT-23, B.Cu at (84.6, 73.1)
- added Q2: MMBT5551-npn, Package_TO_SOT_SMD:SOT-23, B.Cu at (91.0, 73.0)
- added Q3: MMBT5401, Package_TO_SOT_SMD:SOT-23, B.Cu at (120.3, 89.6)
- added Q4: MMBT5551-npn, Package_TO_SOT_SMD:SOT-23, B.Cu at (120.3, 83.1)
- added Q5: MMBT5401, Package_TO_SOT_SMD:SOT-23, B.Cu at (100.1, 72.8)
- added Q6: MMBT5551-npn, Package_TO_SOT_SMD:SOT-23, B.Cu at (106.5, 72.9)
- added Q7: MMBT5401, Package_TO_SOT_SMD:SOT-23, B.Cu at (116.1, 91.9)
- added Q8: MMBT5551-npn, Package_TO_SOT_SMD:SOT-23, B.Cu at (116.1, 83.1)
- added R15: R-1k, Resistor_SMD:R_0805_2012Metric, B.Cu at (96.8, 72.8)
- added R17: R-1k, Resistor_SMD:R_0805_2012Metric, B.Cu at (103.4, 72.8)
- added R18: R-1k, Resistor_SMD:R_0805_2012Metric, B.Cu at (116.5, 95.7)
- added R19: R-1k, Resistor_SMD:R_0805_2012Metric, B.Cu at (116.1, 86.2)
- added R3: R-1k, Resistor_SMD:R_0805_2012Metric, B.Cu at (81.1, 73.0)
- moved R12-10k5 41.4 mm to (88.0, 117.6)
- moved R14 29.9 mm to (120.3, 86.3), turned to 0 degrees
- moved R12 18.4 mm to (120.6, 93.3)
- moved R11-10k1 16.1 mm to (97.0, 95.5), turned to 180 degrees
- moved R4 15.5 mm to (87.8, 73.0), turned to 90 degrees
- moved R12-10k1 15.3 mm to (79.2, 68.5), turned to 90 degrees
- moved R2 15.2 mm to (108.7, 82.9), turned to 90 degrees
- moved Jumper-d6 14.2 mm to (85.2, 81.3)
- moved R1 13.1 mm to (104.6, 81.3), turned to 180 degrees
- moved R6 12.7 mm to (89.0, 82.0), turned to 90 degrees
- moved R12-10k3 11.7 mm to (116.4, 75.6), turned to -90 degrees
- moved R5 10.7 mm to (85.0, 84.0)
- moved R16 10.2 mm to (123.4, 95.7)
- moved Jumper-d5 10.0 mm to (104.6, 84.3)
- moved D5 5.21 mm to (98.3, 89.7)
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Connections:
- J2 pad 2: GNDPWR -> +12C
- J2 pad 3: +12C -> +5C
- J2 pad 4: +5C -> +3.3V
- J2 pad 5: +3.3V -> /mosf1-out-d5
- J2 pad 6: /mosf1-out-d5 -> /mosf2-out-d6
- J2 pad 7: /mosf2-out-d6 -> /mosf3-out-d7
- J2 pad 8: /mosf3-out-d7 -> /d4
- R14 pad 2: /rx -> Net-(Q3-C)
- R4 pad 2: /d0 -> Net-(Q1-C)
Routing:
- net /a0: vias 1 -> 0
- net (no net): vias 2 -> 0

Commit message: update
Parts:
- moved D4 1.09 mm to (99.6, 75.9)
Changed lines of the file:
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@@
 	(footprint "module-custom-for-esp8266:sod80-1n1448"
 		(layer "B.Cu")
-		(at 100.431 76.6)
+		(at 99.6 75.9)
 		(property "Reference" "D4"
 			(at 0.038 0.5 180)

Commit message: update
Parts:
- moved R18 2.50 mm to (118.9, 96.4)
- moved C1 1.58 mm to (99.1, 120.6)
- moved C2 1.58 mm to (81.6, 120.6)
- moved Q2 1.25 mm to (92.1, 72.4)
- moved R6 1.20 mm to (90.0, 82.7)
- moved U3 1.10 mm to (123.6, 120.3)
- moved R4 1.08 mm to (88.7, 72.4)
- moved D2 0.96 mm to (83.8, 75.8)
- moved Q1 0.92 mm to (84.8, 72.2)
- moved R19 0.78 mm to (116.7, 85.7)
- moved IRLR1 0.70 mm to (87.0, 92.6)
- moved U12 0.63 mm to (101.9, 66.0), turned to 90 degrees
- moved R3 0.63 mm to (81.3, 72.4)
- moved U6 0.61 mm to (85.6, 65.7), turned to 90 degrees
- moved Jumper-d6 0.60 mm to (85.0, 81.9)
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- renumbered G*** to G1, G*** to G2, G*** to G3
