File: IoTmanager/topor/IoTmanager_universal.kicad_sch (KiCad schematic)
At the start: 46 parts, among them J1 Conn_01x05_Pin, J2 Conn_01x12_Pin, J3 Conn_01x12_Pin, K1 ZC32F-012-HS3-copy, K2 ZC32F-012-HS3-copy, K3-possible-d1 ZC32F-012-HS3-copy, K4 ZC32F-012-HS3-copy, Q1 BC817, Q2 BC817, Q3 BC817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

Commit message: update
Parts:
- removed J2, J3: Conn_01x12_Pin, module-custom-for-esp8266:connector-12-green-mini, symbol Connector:Conn_01x12_Pin
- removed R3: 100, Resistor_SMD:R_0805_2012Metric, symbol resistor:R-base
- added conn1, conn2: ~, module-custom-for-esp8266:connector-10, symbol models:CONNECTOR-10
- renumbered K3-possible-d1 to K3, Jumper-d5 to R3, Jumper-d6 to R4, Jumper-d7 to R7
Connections:
- net +5C: now also conn1.2
- net GNDPWR: now also conn1.1
- net a0: now also RV1.2
- net conn1-10: now also conn1.10
- net conn1-8: now also conn1.8
- net conn1-9: now also conn1.9
- net conn2-1: now also conn2.1
- net conn2-2: now also conn2.2
- net conn2-3: now also conn2.3
- net conn2-4: now also conn2.4
- net conn2-5: now also conn2.5
- net conn2-6: now also conn2.6
- net conn2-7: now also conn2.7
- net conn2-8: now also conn2.8
- net conn2-9: now also conn2.9
- net d2: now also conn2.10
- net d8: now also conn1.4
- net mosf1-out-d5: now also conn1.5
- net mosf2-out-d6: now also conn1.6
- net mosf3-out-d7: now also conn1.7
- net rx: now also conn1.3
- net at K3.1: now also Q3.3 (C); no longer Q1.3 (C)
- net at R17.1: now also Q3.1 (B); no longer Q1.1 (B)
- net at K2.1: now also Q2.3 (C); no longer Q3.3 (C)
- net at R15.1: now also Q2.1 (B); no longer Q3.1 (B)
- net at K4.1: now also Q4.3 (C); no longer Q2.3 (C)
- net at R14.1: now also Q1.1 (B); no longer Q4.1 (B)
- net at K1.1: now also Q1.3 (C); no longer Q4.3 (C)
- net at R18.1: now also Q4.1 (B); no longer Q2.1 (B)
Other:
- moved on the sheet: K1, K2, R14, R15, R17, R18
